File: pcb/rs485/rs485.sch (KiCad schematic (older format))
At the start: 21 parts

Commit message: Save before autofill
Parts:
- D?: footprint (none) -> rs485:Wickerlib-DIODE-SMC-DO214AB
- J? (x2): footprint (none) -> Socket_Strips:Socket_Strip_Straight_1x02_Pitch2.54mm; Mouser (none) -> NoPart
- J?: footprint (none) -> rs485:Conn-2-8mmx6mm; Mouser (none) -> NoPart
- L?: footprint (none) -> rs485:Inductor-Bourns-SRN8040TA; Mouser (none) -> 652-SRN8040TA-330M
- TP?: footprint (none) -> Measurement_Points:Measurement_Point_Round-SMD-Pad_Small; Mouser (none) -> NoPart
- U?: footprint (none) -> rs485:Exar-NSOIC8
Changed lines of the file:
@@
 F 0 "L?" V 3785 3400 50  0000 C CNN
 F 1 "33uH" V 3694 3400 50  0000 C CNN
-F 2 "" H 3600 3400 50  0001 C CNN
+F 2 "rs485:Inductor-Bourns-SRN8040TA" H 3600 3400 50  0001 C CNN
 F 3 "~" H 3600 3400 50  0001 C CNN
+F 4 "652-SRN8040TA-330M" V 3600 3400 50  0001 C CNN "Mouser"
 	1    3600 3400
 	0    -1   -1   0
@@
 F 0 "D?" V 2604 4218 50  0000 L CNN
 F 1 "VS-MBRS340-M39AT" V 2695 4218 50  0000 L CNN
-F 2 "" V 2650 4150 50  0001 C CNN
+F 2 "rs485:Wickerlib-DIODE-SMC-DO214AB" V 2650 4150 50  0001 C CNN
 F 3 "~" V 2650 4150 50  0001 C CNN
 F 4 "78-VS-MBRS340-M39AT" V 2650 4150 50  0001 C CNN "Mouser"
@@
 F 0 "U?" H 7375 3465 50  0000 C CNN
 F 1 "SP485CN-L_TR" H 7375 3374 50  0000 C CNN
-F 2 "" H 7350 3400 50  0001 C CNN
+F 2 "rs485:Exar-NSOIC8" H 7350 3400 50  0001 C CNN
 F 3 "" H 7350 3400 50  0001 C CNN
 F 4 "701-SP485CN-L/TR" H 7350 3400 50  0001 C CNN "Mouser"
@@
 F 0 "J?" H 8480 3692 50  0000 L CNN
 F 1 "Conn_01x02" H 8480 3601 50  0000 L CNN
-F 2 "" H 8400 3700 50  0001 C CNN
+F 2 "Socket_Strips:Socket_Strip_Straight_1x02_Pitch2.54mm" H 8400 3700 50  0001 C CNN
 F 3 "~" H 8400 3700 50  0001 C CNN
+F 4 "NoPart" H 8400 3700 50  0001 C CNN "Mouser"
 	1    8400 3700
 	1    0    0    -1
@@
 F 0 "J?" H 8480 3992 50  0000 L CNN
 F 1 "Conn_01x02" H 8480 3901 50  0000 L CNN
-F 2 "" H 8400 4000 50  0001 C CNN
+F 2 "Socket_Strips:Socket_Strip_Straight_1x02_Pitch2.54mm" H 8400 4000 50  0001 C CNN
 F 3 "~" H 8400 4000 50  0001 C CNN
+F 4 "NoPart" H 8400 4000 50  0001 C CNN "Mouser"
 	1    8400 4000
 	1    0    0    -1
@@
 F 0 "J?" H 2070 3867 50  0000 C CNN
 F 1 "Power" H 2070 3776 50  0000 C CNN
-F 2 "" H 2150 3650 50  0001 C CNN
+F 2 "rs485:Conn-2-8mmx6mm" H 2150 3650 50  0001 C CNN
 F 3 "~" H 2150 3650 50  0001 C CNN
+F 4 "NoPart" H 2150 3650 50  0001 C CNN "Mouser"
 	1    2150 3650
 	-1   0    0    -1
@@
 F 0 "TP?" H 5358 3370 50  0000 L CNN
 F 1 "TestPoint" H 5358 3279 50  0000 L CNN
-F 2 "" H 5500 3250 50  0001 C CNN
+F 2 "Measurement_Points:Measurement_Point_Round-SMD-Pad_Small" H 5500 3250 50  0001 C CNN
 F 3 "~" H 5500 3250 50  0001 C CNN
+F 4 "NoPart" H 5300 3250 50  0001 C CNN "Mouser"
 	1    5300 3250
 	1    0    0    -1

Commit message: Finish layout
Parts:
- removed J?: Conn_01x04, Socket_Strips:Socket_Strip_Straight_1x04_Pitch2.54mm, symbol Connector_Generic:Conn_01x04
- added C3, C6: 10uF, Capacitors_SMD:CP_Elec_5x5.7, symbol Device:C_Small
- added C5: 47uF, Capacitors_SMD:CP_Elec_6.3x5.8, symbol Device:C_Small
- added J2: Conn_01x05, Socket_Strips:Socket_Strip_Straight_1x05_Pitch2.54mm, symbol Connector_Generic:Conn_01x05
- added MH1, MH2, MH3, MH4: MountingHole, Mounting_Holes:MountingHole_5.3mm_M5, symbol Mechanical:MountingHole
- C2: renamed from C?; footprint Capacitors_SMD:CP_Elec_6.3x5.3 -> Capacitors_SMD:CP_Elec_5x5.3; Mouser 140-VE101M1CTR0605 -> 710-875105242010
- C7: renamed from C?; value 1.5nF -> 2.2nF; Mouser 77-VJ0402Y152KXAPBC -> 710-885012205027
- R5: renamed from R?; Mouser 603-AC0603JR-0712KL -> 603-AC0402JR-078K2L
- TP2, TP3: renamed from TP?; footprint (none) -> Measurement_Points:Measurement_Point_Round-SMD-Pad_Small; Mouser (none) -> NoPart
- gave numbers to parts that had none: 15
Connections:
- wire segments 69 -> 88

Commit message: Generate BOMs
Other:
- note added: "DNP; there's already an inherent pulldown in the IC"
Changed lines of the file:
@@
 Wire Wire Line
 	8650 3800 8400 3800
-Text Notes 8700 4300 0    50   ~ 0
+Text Notes 8950 3350 0    50   ~ 0
 Second one's for daisy chaining them
 Text Label 5600 5100 0    50   ~ 0
@@
 Wire Wire Line
 	6800 4000 6800 4100
+Text Notes 7700 4350 0    50   ~ 0
+DNP; there's already an inherent pulldown in the IC
 $EndSCHEMATC
