File: pcb/peripherals/peripherals.kicad_pcb (KiCad board)
At the start: 2 copper layers, 113.5 x 124.5 mm, 134 parts, among them J101 Conn_01x05, J102 Conn_01x05, J103 Conn_01x04, J104 Conn_01x04, J105 Conn_01x04, J106 Conn_01x04, J107 Conn_01x05, J108 Conn_01x05, Q201 RQ3E100BNTB, Q202 RQ3E100BNTB, Q301 RQ3E100BNTB, Q302 RQ3E100BNTB, Q401 RQ3E100BNTB, Q402 RQ3E100BNTB, Q501 RQ3E100BNTB, Q502 RQ3E100BNTB, Q601 RQ3E100BNTB, Q602 RQ3E100BNTB, Q701 RQ3E100BNTB, Q702 RQ3E100BNTB, Q801 RQ3E100BNTB, Q802 RQ3E100BNTB, Q901 RQ3E100BNTB, Q902 RQ3E100BNTB, U201 DGD0506A, U301 DGD0506A, U401 DGD0506A, U501 DGD0506A, U601 DGD0506A, U701 DGD0506A, U801 DGD0506A, U901 DGD0506A

Commit message: Save before autotile
Parts:
- removed C203, C303, C403, C503, C603, C703, C803, C903: 470uF, Capacitors_ThroughHole:CP_Radial_D10.0mm_P5.00mm
- removed C204, C304, C404, C504, C604, C704, C804, C904: 1000uF, Capacitors_ThroughHole:CP_Radial_D18.0mm_P7.50mm
- added C101: 470uF, Capacitors_ThroughHole:CP_Radial_D10.0mm_P5.00mm, F.Cu at (214.3, 50.2)
- added C102: 470uF, Capacitors_ThroughHole:CP_Radial_D10.0mm_P5.00mm, F.Cu at (214.3, 61.0)
- added C103: 1000uF, Capacitors_ThroughHole:CP_Radial_D18.0mm_P7.50mm, F.Cu at (188.1, 40.4)
- added C104: 1000uF, Capacitors_ThroughHole:CP_Radial_D18.0mm_P7.50mm, F.Cu at (169.4, 40.4)
- J103, J104: footprint peripherals:Conn-4-8mmx6mm -> peripherals:Conn-4-8mmx3mm
- J105, J106: footprint peripherals:Conn-4-8mmx6mm -> peripherals:Conn-4-8mmx3mm; moved to F.Cu
- moved Q401 209.9 mm to (245.3, 33.4), turned to 0 degrees
- moved TP401 209.0 mm to (247.6, 36.4)
- moved TP402 208.8 mm to (244.5, 37.9)
- moved Q402 207.9 mm to (240.5, 35.2), turned to 0 degrees
- moved R401 204.8 mm to (244.6, 36.1)
- moved TP202 203.5 mm to (259.3, 73.9)
- moved R403 202.7 mm to (239.4, 38.0), turned to 0 degrees
- moved R402 202.5 mm to (246.3, 38.0), turned to 0 degrees
- moved Q201 201.1 mm to (257.0, 70.9), turned to 0 degrees
- moved C405 200.9 mm to (242.4, 38.8), turned to 0 degrees
- moved C406 199.1 mm to (239.3, 39.4), turned to 0 degrees
- moved C402 196.6 mm to (242.4, 37.8)
- moved Q202 196.2 mm to (252.2, 72.8), turned to 0 degrees
- moved R201 196.1 mm to (256.3, 73.6)
- moved TP201 194.7 mm to (254.1, 76.9)
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Routing:
- net GND: track 823.6 -> 18.3 mm, vias 63 -> 4
- net +BATT: track 418.8 -> 5.98 mm
- net /sheet5B6E69C4/IN: track 71.6 -> 0.00 mm, vias 2 -> 0
- net /sheet5B6E69C4/EN: track 68.3 -> 0.00 mm, vias 2 -> 0
- net /sheet5B6E6A5D/EN: track 65.3 -> 0.00 mm, vias 3 -> 0
- net /sheet5B6E6A5D/IN: track 62.9 -> 0.00 mm, vias 3 -> 0
- net /Sheet5B7230C3/OUT: track 56.1 -> 0.00 mm
- net /sheet5B6E6A5A/IN: track 55.5 -> 0.00 mm, vias 2 -> 0
- net /sheet5B6E6A5A/EN: track 55.4 -> 0.00 mm, vias 2 -> 0
- net /Sheet5B7230C3/EN: track 53.9 -> 0.00 mm, vias 3 -> 0
- net /Sheet5B7230C3/IN: track 53.6 -> 0.00 mm, vias 3 -> 0
- net /sheet5B6E6A5D/OUT: track 51.2 -> 0.00 mm
- net /sheet5B6E69C3/IN: track 40.5 -> 0.00 mm, vias 3 -> 0
- net /sheet5B6E6A5C/EN: track 39.8 -> 0.00 mm, vias 3 -> 0
- net /sheet5B6E69C3/EN: track 39.8 -> 0.00 mm, vias 1 -> 0
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- removed copper zone on F.Cu, net +BATT
- removed copper zone on F.Cu, net /Sheet5B7230C3/OUT
- removed copper zone on F.Cu, net /sheet5B6E69B5/OUT
- removed copper zone on F.Cu, net /sheet5B6E69C3/OUT
- removed copper zone on F.Cu, net /sheet5B6E69C4/OUT
- removed copper zone on F.Cu, net /sheet5B6E6A5A/OUT
- removed copper zone on F.Cu, net /sheet5B6E6A5B/OUT
- removed copper zone on F.Cu, net /sheet5B6E6A5C/OUT
- removed copper zone on F.Cu, net /sheet5B6E6A5D/OUT
- removed copper zone on B.Cu, net GND
- removed copper zone on F.Cu, net GND
