File: pcb/receiver/receiver.sch (KiCad schematic (older format))
At the start: 0 parts

Commit message: Work out signal processing and power sections TODO MCU stuff
Parts:
- added C101, C104, C115, C117: 10 uF, symbol Device:C_Small
- added C102: 4.7 nF, symbol Device:C_Small
- added C103, C105, C110, C111: 0.1 uF, symbol Device:C_Small
- added C106, C108, C109, C113, C114, C116: 4.7 uF, symbol Device:C_Small
- added C107: 1 nF, symbol Device:C_Small
- added C112: 10 pF, symbol Device:C_Small
- added D101, D102: D_Schottky_Small, symbol Device:D_Schottky_Small
- added L101: 47 uH, symbol Device:L_Small
- added L102: 10 uH, symbol Device:L_Small
- added Q101: Q_PMOS_DSG, symbol Device:Q_PMOS_DSG
- added R101: 10, symbol Device:R_Small
- added R102: 680k, symbol Device:R_Small
- added R103: 47k, symbol Device:R_Small
- added R104: 120k, symbol Device:R_Small
- added R105: 1.2M, symbol Device:R_Small
- added R106: 100k, symbol Device:R_Small
- added U101: TPS63700DRCR, symbol receiver:TPS63700DRCR
- added U102: NCP1403SNT1G, symbol receiver:NCP1403SNT1G
Connections:
- new net: C102.1, U101.1 (COMP)
- new net: C110.1, C111.1, R104.1, U101.10 (VREF)
- new net: C103.1, R101.2, U101.3 (VIN), U101.4 (EN)
- new net: D102.1 (K), L102.1, U101.6 (SW)
- new net: C112.1, R104.2, R105.1, U101.9 (FB)
- new net: C112.2, R106.1
- new net: C107.2, R102.2, R103.1, U102.2 (FB)
- new net: D101.2 (A), L101.2, U102.5 (LX)
- new net +12V: C107.1, C108.1, C113.1, C115.1, C117.1, D101.1 (K), R102.1
- new net +5V_DIGITAL: C101.1, C104.1, C105.1, L101.1, Q101.2 (S), R101.1, U101.5 (IN), U102.1 (CE), U102.3 (VDD)
- new net +5V_INPUT: Q101.1 (D)
- new net -12V: C106.1, C109.1, C114.1, C116.1, D102.2 (A), R105.2, R106.2, U101.8 (OUT)
- new net GND: C101.2, C102.2, C103.2, C104.2, C105.2, C106.2, C108.2, C109.2, C110.2, C111.2, C113.2, C114.2, C115.2, C116.2, C117.2, L102.2, Q101.3 (G), R103.2, U101.11 (GPAD), U101.2 (GND), U101.7 (PS_GND), U102.4 (GND)
Other:
- note added: "TODO footprint"
- note added: "TODO source schottky diode"
