File: pcb/receiver/receiver.sch (KiCad schematic (older format))
At the start: 30 parts, among them Q101 Q_PMOS_DSG, U101 TPS63700DRCR, U102 NCP1403SNT1G

Commit message: Add all components TODO footprint/source everything
Parts:
- added J101: Conn_01x02, symbol Connector_Generic:Conn_01x02
- added Q102: Q_NPN_BCE, symbol Device:Q_NPN_BCE
- added Q103: Q_PMOS_DSG, symbol Device:Q_PMOS_DSG
- added R107: 1k, symbol Device:R_Small
- added R108: 100k, symbol Device:R_Small
- D101, D102: value D_Schottky_Small -> 2SS100L-W
Connections:
- net GND: now also J101.1 (Pin_1), Q102.3 (E)
- net +5V_DIGITAL renamed +5V
- net +5V: now also Q103.1 (D); no longer Q101.2 (S)
- net +5V_INPUT: no longer names the net of Q101.1 (D)
- net +5V_INPUT: now also J101.2 (Pin_2)
- new net: Q102.2 (C), Q103.3 (G), R108.2
- new net: Q102.1 (B), R107.1
- new net +5V_USB: Q101.2 (S), Q103.2 (S), R108.1
- new net ANALOG_EN: R107.2
Other:
- note removed: "TODO source schottky diode"
- moved on the sheet: C101, C102, C103, C104, C105, C106, C107, C108, C109, C110, C111, C112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

Commit message: Most parts footprinted; TODO analog voltage reference, photodiodes, passives
Parts:
- U101: footprint (none) -> receiver-footprints:TI-VSON10; Mouser (none) -> 595-TPS63700DRCR
- U102: footprint (none) -> receiver-footprints:ON-TSOP-5
Other:
- note removed: "TODO footprint"
Changed lines of the file:
@@
 F 0 "U101" H 2500 6250 50  0000 C CNN
 F 1 "TPS63700DRCR" H 2550 5350 50  0000 C CNN
-F 2 "" H 2500 6250 50  0001 C CNN
+F 2 "receiver-footprints:TI-VSON10" H 2500 6250 50  0001 C CNN
 F 3 "" H 2500 6250 50  0001 C CNN
+F 4 "595-TPS63700DRCR" H 2500 6250 50  0001 C CNN "Mouser"
 	1    2500 6250
 	1    0    0    -1
@@
 Wire Wire Line
 	4300 5800 4500 5800
-Text Notes 2300 7350 0    50   ~ 0
-TODO footprint
 $Comp
 L receiver:NCP1403SNT1G U102
@@
 F 0 "U102" H 3800 4850 50  0000 C CNN
 F 1 "NCP1403SNT1G" H 3800 4450 50  0000 C CNN
-F 2 "" H 3700 4850 50  0001 C CNN
+F 2 "receiver-footprints:ON-TSOP-5" H 3700 4850 50  0001 C CNN
 F 3 "" H 3700 4850 50  0001 C CNN
 	1    3800 4650

Commit message: Source most passives; save before autofill
Parts:
- removed Q102: Q_NPN_BCE, symbol Device:Q_NPN_BCE
- added Q?: MMBT2222A-7-F, symbol Device:Q_NPN_BEC
- C103, C105, C110, C111: value 0.1 uF -> 100 nF
- C108: footprint (none) -> Capacitors_SMD:CP_Elec_4x5.3; Mouser (none) -> 647-UWX1E4R7MCL1
- C112: footprint (none) -> Capacitors_SMD:C_0402; Mouser (none) -> 710-885012005074
- R102: footprint (none) -> Resistors_SMD:R_0603_HandSoldering; Mouser (none) -> 603-RC0603FR-13680KL
- R103: footprint (none) -> Resistors_SMD:R_0603_HandSoldering; Mouser (none) -> 603-RC0603FR-0747KL
- R104: footprint (none) -> Resistors_SMD:R_0603_HandSoldering; Mouser (none) -> 603-RC0603FR-07120KL
- R105: footprint (none) -> Resistors_SMD:R_0402; Mouser (none) -> 603-RC0402JR-071M2L
- U102: Mouser (none) -> 863-NCP1403SNT1G
Connections:
- net GND: now also Q?.2 (E)
- net at Q103.3 (G), R108.2: now also Q?.3 (C)
- net at R107.1: now also Q?.1 (B)
Changed lines of the file:
@@
 P 1950 7000
 F 0 "C103" H 1960 7070 50  0000 L CNN
-F 1 "0.1 uF" H 1960 6920 50  0000 L CNN
+F 1 "100 nF" H 1960 6920 50  0000 L CNN
 F 2 "" H 1950 7000 50  0001 C CNN
 F 3 "~" H 1950 7000 50  0001 C CNN
@@
 F 0 "R105" H 3980 6620 50  0000 L CNN
 F 1 "1.2M" H 3980 6560 50  0000 L CNN
-F 2 "" H 3950 6600 50  0001 C CNN
+F 2 "Resistors_SMD:R_0402" H 3950 6600 50  0001 C CNN
 F 3 "~" H 3950 6600 50  0001 C CNN
+F 4 "603-RC0402JR-071M2L" H 3950 6600 50  0001 C CNN "Mouser"
 	1    3950 6600
 	1    0    0    -1
@@
 F 0 "R104" H 3980 6320 50  0000 L CNN
 F 1 "120k" H 3980 6260 50  0000 L CNN
-F 2 "" H 3950 6300 50  0001 C CNN
+F 2 "Resistors_SMD:R_0603_HandSoldering" H 3950 6300 50  0001 C CNN
 F 3 "~" H 3950 6300 50  0001 C CNN
+F 4 "603-RC0603FR-07120KL" H 3950 6300 50  0001 C CNN "Mouser"
 	1    3950 6300
 	1    0    0    -1
@@
 F 0 "C112" H 4310 6520 50  0000 L CNN
 F 1 "10 pF" H 4310 6370 50  0000 L CNN
-F 2 "" H 4300 6450 50  0001 C CNN
+F 2 "Capacitors_SMD:C_0402" H 4300 6450 50  0001 C CNN
 F 3 "~" H 4300 6450 50  0001 C CNN
+F 4 "710-885012005074" H 4300 6450 50  0001 C CNN "Mouser"
 	1    4300 6450
 	0    -1   -1   0
@@
 P 4200 6100
 F 0 "C111" H 4210 6170 50  0000 L CNN
-F 1 "0.1 uF" H 4210 6020 50  0000 L CNN
+F 1 "100 nF" H 4210 6020 50  0000 L CNN
 F 2 "" H 4200 6100 50  0001 C CNN
 F 3 "~" H 4200 6100 50  0001 C CNN
@@
 P 4200 5800
 F 0 "C110" H 4210 5870 50  0000 L CNN
-F 1 "0.1 uF" H 4210 5720 50  0000 L CNN
+F 1 "100 nF" H 4210 5720 50  0000 L CNN
 F 2 "" H 4200 5800 50  0001 C CNN
 F 3 "~" H 4200 5800 50  0001 C CNN
@@
 F 2 "receiver-footprints:ON-TSOP-5" H 3700 4850 50  0001 C CNN
 F 3 "" H 3700 4850 50  0001 C CNN
+F 4 "863-NCP1403SNT1G" H 3800 4650 50  0001 C CNN "Mouser"
 	1    3800 4650
 	1    0    0    -1
@@
 F 0 "C108" H 5010 4620 50  0000 L CNN
 F 1 "4.7 uF" H 5010 4470 50  0000 L CNN
-F 2 "" H 5000 4550 50  0001 C CNN
+F 2 "Capacitors_SMD:CP_Elec_4x5.3" H 5000 4550 50  0001 C CNN
 F 3 "~" H 5000 4550 50  0001 C CNN
+F 4 "647-UWX1E4R7MCL1" H 5000 4550 50  0001 C CNN "Mouser"
 	1    5000 4550
 	1    0    0    -1
@@
 F 0 "R102" H 4430 4720 50  0000 L CNN
 F 1 "680k" H 4430 4660 50  0000 L CNN
-F 2 "" H 4400 4700 50  0001 C CNN
+F 2 "Resistors_SMD:R_0603_HandSoldering" H 4400 4700 50  0001 C CNN
 F 3 "~" H 4400 4700 50  0001 C CNN
+F 4 "603-RC0603FR-13680KL" H 4400 4700 50  0001 C CNN "Mouser"
 	1    4400 4700
 	1    0    0    -1
@@
 F 0 "R103" H 4430 5120 50  0000 L CNN
 F 1 "47k" H 4430 5060 50  0000 L CNN
-F 2 "" H 4400 5100 50  0001 C CNN
+F 2 "Resistors_SMD:R_0603_HandSoldering" H 4400 5100 50  0001 C CNN
 F 3 "~" H 4400 5100 50  0001 C CNN
+F 4 "603-RC0603FR-0747KL" H 4400 5100 50  0001 C CNN "Mouser"
 	1    4400 5100
 	1    0    0    -1
@@
 P 3200 4950
 F 0 "C105" H 3210 5020 50  0000 L CNN
-F 1 "0.1 uF" H 3210 4870 50  0000 L CNN
+F 1 "100 nF" H 3210 4870 50  0000 L CNN
 F 2 "" H 3200 4950 50  0001 C CNN
 F 3 "~" H 3200 4950 50  0001 C CNN
@@
 Wire Wire Line
 	2650 5050 2650 4850
-$Comp
-L Device:Q_NPN_BCE Q102
-U 1 1 5C340CBF
-P 2200 5350
-F 0 "Q102" H 2400 5400 50  0000 L CNN
-F 1 "Q_NPN_BCE" H 2400 5300 50  0000 L CNN
-F 2 "" H 2400 5450 50  0001 C CNN
-F 3 "~" H 2200 5350 50  0001 C CNN
-	1    2200 5350
-	1    0    0    -1
-$EndComp
 Wire Wire Line
 	2300 5050 2300 5150
@@
 Wire Wire Line
 	1950 6850 1950 6900
+$Comp
+L Device:Q_NPN_BEC Q?
+U 1 1 5C66C411
+P 2200 5350
+F 0 "Q?" H 2400 5400 50  0000 L CNN
+F 1 "MMBT2222A-7-F" H 2400 5300 50  0000 L CNN
+F 2 "" H 2400 5450 50  0001 C CNN
+F 3 "~" H 2200 5350 50  0001 C CNN
+	1    2200 5350
+	1    0    0    -1
+$EndComp
 $EndSCHEMATC

Commit message: Autofill components
Parts:
- C101, C104, C115, C117: footprint (none) -> Capacitors_SMD:C_0805_HandSoldering; Mouser (none) -> 81-GRM21BR61E106MA3L
- C103, C105, C110, C111: footprint (none) -> Capacitors_SMD:C_0603_HandSoldering; Mouser (none) -> 710-885012206071
- C106, C109, C113, C114, C116: footprint (none) -> Capacitors_SMD:CP_Elec_4x5.3; Mouser (none) -> 647-UWX1E4R7MCL1
- C107: footprint (none) -> Capacitors_SMD:C_0402; Mouser (none) -> 710-885012205061
- Q?: footprint (none) -> TO_SOT_Packages_SMD:SOT-23_Handsoldering; Mouser (none) -> 621-MMBT2222A-F
- R106, R108: footprint (none) -> Resistors_SMD:R_0402; Mouser (none) -> 603-RC0402JR-13100KL
- R107: footprint (none) -> Resistors_SMD:R_0603_HandSoldering; Mouser (none) -> 603-RC0603JR-071KL
Changed lines of the file:
@@
 F 0 "C101" H 1660 7070 50  0000 L CNN
 F 1 "10 uF" H 1660 6920 50  0000 L CNN
-F 2 "" H 1650 7000 50  0001 C CNN
+F 2 "Capacitors_SMD:C_0805_HandSoldering" H 1650 7000 50  0001 C CNN
 F 3 "~" H 1650 7000 50  0001 C CNN
+F 4 "81-GRM21BR61E106MA3L" H 1650 7000 50  0001 C CNN "Mouser"
 	1    1650 7000
 	-1   0    0    -1
@@
 F 0 "C103" H 1960 7070 50  0000 L CNN
 F 1 "100 nF" H 1960 6920 50  0000 L CNN
-F 2 "" H 1950 7000 50  0001 C CNN
+F 2 "Capacitors_SMD:C_0603_HandSoldering" H 1950 7000 50  0001 C CNN
 F 3 "~" H 1950 7000 50  0001 C CNN
+F 4 "710-885012206071" H 1950 7000 50  0001 C CNN "Mouser"
 	1    1950 7000
 	-1   0    0    -1
@@
 F 0 "C106" H 3760 7070 50  0000 L CNN
 F 1 "4.7 uF" H 3760 6920 50  0000 L CNN
-F 2 "" H 3750 7000 50  0001 C CNN
+F 2 "Capacitors_SMD:CP_Elec_4x5.3" H 3750 7000 50  0001 C CNN
 F 3 "~" H 3750 7000 50  0001 C CNN
+F 4 "647-UWX1E4R7MCL1" H 3750 7000 50  0001 C CNN "Mouser"
 	1    3750 7000
 	1    0    0    -1
@@
 F 0 "C109" H 4160 7070 50  0000 L CNN
 F 1 "4.7 uF" H 4160 6920 50  0000 L CNN
-F 2 "" H 4150 7000 50  0001 C CNN
+F 2 "Capacitors_SMD:CP_Elec_4x5.3" H 4150 7000 50  0001 C CNN
 F 3 "~" H 4150 7000 50  0001 C CNN
+F 4 "647-UWX1E4R7MCL1" H 4150 7000 50  0001 C CNN "Mouser"
 	1    4150 7000
 	1    0    0    -1
@@
 F 0 "C114" H 4510 7070 50  0000 L CNN
 F 1 "4.7 uF" H 4510 6920 50  0000 L CNN
-F 2 "" H 4500 7000 50  0001 C CNN
+F 2 "Capacitors_SMD:CP_Elec_4x5.3" H 4500 7000 50  0001 C CNN
 F 3 "~" H 4500 7000 50  0001 C CNN
+F 4 "647-UWX1E4R7MCL1" H 4500 7000 50  0001 C CNN "Mouser"
 	1    4500 7000
 	1    0    0    -1
@@
 F 0 "C116" H 4860 7070 50  0000 L CNN
 F 1 "4.7 uF" H 4860 6920 50  0000 L CNN
-F 2 "" H 4850 7000 50  0001 C CNN
+F 2 "Capacitors_SMD:CP_Elec_4x5.3" H 4850 7000 50  0001 C CNN
 F 3 "~" H 4850 7000 50  0001 C CNN
+F 4 "647-UWX1E4R7MCL1" H 4850 7000 50  0001 C CNN "Mouser"
 	1    4850 7000
 	1    0    0    -1
@@
 F 0 "R106" H 4680 6620 50  0000 L CNN
 F 1 "100k" H 4680 6560 50  0000 L CNN
-F 2 "" H 4650 6600 50  0001 C CNN
+F 2 "Resistors_SMD:R_0402" H 4650 6600 50  0001 C CNN
 F 3 "~" H 4650 6600 50  0001 C CNN
+F 4 "603-RC0402JR-13100KL" H 4650 6600 50  0001 C CNN "Mouser"
 	1    4650 6600
 	1    0    0    -1
@@
 F 0 "C111" H 4210 6170 50  0000 L CNN
 F 1 "100 nF" H 4210 6020 50  0000 L CNN
-F 2 "" H 4200 6100 50  0001 C CNN
+F 2 "Capacitors_SMD:C_0603_HandSoldering" H 4200 6100 50  0001 C CNN
 F 3 "~" H 4200 6100 50  0001 C CNN
+F 4 "710-885012206071" H 4200 6100 50  0001 C CNN "Mouser"
 	1    4200 6100
 	0    -1   -1   0
@@
 F 0 "C110" H 4210 5870 50  0000 L CNN
 F 1 "100 nF" H 4210 5720 50  0000 L CNN
-F 2 "" H 4200 5800 50  0001 C CNN
+F 2 "Capacitors_SMD:C_0603_HandSoldering" H 4200 5800 50  0001 C CNN
 F 3 "~" H 4200 5800 50  0001 C CNN
+F 4 "710-885012206071" H 4200 5800 50  0001 C CNN "Mouser"
 	1    4200 5800
 	0    -1   -1   0
@@
 F 0 "C113" H 5410 4620 50  0000 L CNN
 F 1 "4.7 uF" H 5410 4470 50  0000 L CNN
-F 2 "" H 5400 4550 50  0001 C CNN
+F 2 "Capacitors_SMD:CP_Elec_4x5.3" H 5400 4550 50  0001 C CNN
 F 3 "~" H 5400 4550 50  0001 C CNN
+F 4 "647-UWX1E4R7MCL1" H 5400 4550 50  0001 C CNN "Mouser"
 	1    5400 4550
 	1    0    0    -1
@@
 F 0 "C115" H 5760 4620 50  0000 L CNN
 F 1 "10 uF" H 5760 4470 50  0000 L CNN
-F 2 "" H 5750 4550 50  0001 C CNN
+F 2 "Capacitors_SMD:C_0805_HandSoldering" H 5750 4550 50  0001 C CNN
 F 3 "~" H 5750 4550 50  0001 C CNN
+F 4 "81-GRM21BR61E106MA3L" H 5750 4550 50  0001 C CNN "Mouser"
 	1    5750 4550
 	1    0    0    -1
@@
 F 0 "C117" H 6110 4620 50  0000 L CNN
 F 1 "10 uF" H 6110 4470 50  0000 L CNN
-F 2 "" H 6100 4550 50  0001 C CNN
+F 2 "Capacitors_SMD:C_0805_HandSoldering" H 6100 4550 50  0001 C CNN
 F 3 "~" H 6100 4550 50  0001 C CNN
+F 4 "81-GRM21BR61E106MA3L" H 6100 4550 50  0001 C CNN "Mouser"
 	1    6100 4550
 	1    0    0    -1
@@
 F 0 "C107" H 4810 4770 50  0000 L CNN
 F 1 "1 nF" H 4810 4620 50  0000 L CNN
-F 2 "" H 4800 4700 50  0001 C CNN
+F 2 "Capacitors_SMD:C_0402" H 4800 4700 50  0001 C CNN
 F 3 "~" H 4800 4700 50  0001 C CNN
+F 4 "710-885012205061" H 4800 4700 50  0001 C CNN "Mouser"
 	1    4800 4700
 	1    0    0    -1
@@
 F 0 "C104" H 3060 5020 50  0000 L CNN
 F 1 "10 uF" H 3060 4870 50  0000 L CNN
-F 2 "" H 3050 4950 50  0001 C CNN
+F 2 "Capacitors_SMD:C_0805_HandSoldering" H 3050 4950 50  0001 C CNN
 F 3 "~" H 3050 4950 50  0001 C CNN
+F 4 "81-GRM21BR61E106MA3L" H 3050 4950 50  0001 C CNN "Mouser"
 	1    3050 4950
 	-1   0    0    -1
@@
 F 0 "C105" H 3210 5020 50  0000 L CNN
 F 1 "100 nF" H 3210 4870 50  0000 L CNN
-F 2 "" H 3200 4950 50  0001 C CNN
+F 2 "Capacitors_SMD:C_0603_HandSoldering" H 3200 4950 50  0001 C CNN
 F 3 "~" H 3200 4950 50  0001 C CNN
+F 4 "710-885012206071" H 3200 4950 50  0001 C CNN "Mouser"
 	1    3200 4950
 	1    0    0    -1
@@
 F 0 "R108" H 2330 4820 50  0000 L CNN
 F 1 "100k" H 2330 4760 50  0000 L CNN
-F 2 "" H 2300 4800 50  0001 C CNN
+F 2 "Resistors_SMD:R_0402" H 2300 4800 50  0001 C CNN
 F 3 "~" H 2300 4800 50  0001 C CNN
+F 4 "603-RC0402JR-13100KL" H 2300 4800 50  0001 C CNN "Mouser"
 	1    2300 4800
 	-1   0    0    -1
@@
 F 0 "R107" H 1830 5370 50  0000 L CNN
 F 1 "1k" H 1830 5310 50  0000 L CNN
-F 2 "" H 1800 5350 50  0001 C CNN
+F 2 "Resistors_SMD:R_0603_HandSoldering" H 1800 5350 50  0001 C CNN
 F 3 "~" H 1800 5350 50  0001 C CNN
+F 4 "603-RC0603JR-071KL" H 1800 5350 50  0001 C CNN "Mouser"
 	1    1800 5350
 	0    1    1    0
@@
 F 0 "Q?" H 2400 5400 50  0000 L CNN
 F 1 "MMBT2222A-7-F" H 2400 5300 50  0000 L CNN
-F 2 "" H 2400 5450 50  0001 C CNN
+F 2 "TO_SOT_Packages_SMD:SOT-23_Handsoldering" H 2400 5450 50  0001 C CNN
 F 3 "~" H 2200 5350 50  0001 C CNN
+F 4 "621-MMBT2222A-F" H 2200 5350 50  0001 C CNN "Mouser"
 	1    2200 5350
 	1    0    0    -1

Commit message: Footprint more stuff
Parts:
- removed Q101, Q103: Q_PMOS_DSG, symbol Device:Q_PMOS_DSG
- added D103: 2SS100L-W, symbol Device:D_Schottky_Small
- added Q?: BSS215PH6327XTSA1, TO_SOT_Packages_SMD:SOT-23_Handsoldering, symbol Device:Q_PMOS_GSD
- C102: footprint (none) -> Capacitors_SMD:C_0402; Mouser (none) -> 710-885012205029
- L101: footprint (none) -> Capacitors_SMD:C_0805_HandSoldering; Mouser (none) -> 810-MLZ2012M470WT000
- L102: footprint (none) -> Capacitors_SMD:C_0805_HandSoldering; Mouser (none) -> 810-MLZ2012M100WT000
- R101: footprint (none) -> Capacitors_SMD:C_0402; Mouser (none) -> 667-ERJ-U02D10R0X
- gave numbers to parts that had none: 1
Connections:
- net +5V: now also Q?.3 (D)
- net +5V_USB: now also D103.1 (K), Q?.2 (S)
- net at Q102.3 (C), R108.2: now also Q?.1 (G)
- net at J101.2 (Pin_2): now also D103.2 (A)
Other:
- moved on the sheet: J101
Changed lines of the file:
@@
 -12V
 Wire Wire Line
-	1600 4550 1300 4550
-$Comp
-L Device:Q_PMOS_DSG Q101
-U 1 1 5D19B343
-P 1800 4650
-F 0 "Q101" H 2000 4700 50  0000 L CNN
-F 1 "Q_PMOS_DSG" H 2000 4600 50  0000 L CNN
-F 2 "" H 2000 4750 50  0001 C CNN
-F 3 "~" H 1800 4650 50  0001 C CNN
-	1    1800 4650
-	0    -1   -1   0
-$EndComp
-Wire Wire Line
 	2100 4550 2100 4450
-$Comp
-L power:GND #PWR0104
-U 1 1 5D19B3DE
-P 1800 4950
-F 0 "#PWR0104" H 1800 4700 50  0001 C CNN
-F 1 "GND" H 1800 4800 50  0000 C CNN
-F 2 "" H 1800 4950 50  0001 C CNN
-F 3 "" H 1800 4950 50  0001 C CNN
-	1    1800 4950
-	1    0    0    -1
-$EndComp
-Wire Wire Line
-	1800 4850 1800 4950
 $Comp
 L receiver:TPS63700DRCR U101
@@
 F 0 "R101" H 1830 6620 50  0000 L CNN
 F 1 "10" H 1830 6560 50  0000 L CNN
-F 2 "" H 1800 6600 50  0001 C CNN
+F 2 "Capacitors_SMD:C_0402" H 1800 6600 50  0001 C CNN
 F 3 "~" H 1800 6600 50  0001 C CNN
+F 4 "667-ERJ-U02D10R0X" H 1800 6600 50  0001 C CNN "Mouser"
 	1    1800 6600
 	0    -1   1    0
@@
 F 0 "L102" H 3280 7040 50  0000 L CNN
 F 1 "10 uH" H 3280 6960 50  0000 L CNN
-F 2 "" H 3250 7000 50  0001 C CNN
+F 2 "Capacitors_SMD:C_0805_HandSoldering" H 3250 7000 50  0001 C CNN
 F 3 "~" H 3250 7000 50  0001 C CNN
+F 4 "810-MLZ2012M100WT000" H 3250 7000 50  0001 C CNN "Mouser"
 	1    3250 7000
 	1    0    0    -1
@@
 F 0 "C102" H 1810 6370 50  0000 L CNN
 F 1 "4.7 nF" H 1810 6220 50  0000 L CNN
-F 2 "" H 1800 6300 50  0001 C CNN
+F 2 "Capacitors_SMD:C_0402" H 1800 6300 50  0001 C CNN
 F 3 "~" H 1800 6300 50  0001 C CNN
+F 4 "710-885012205029" H 1800 6300 50  0001 C CNN "Mouser"
 	1    1800 6300
 	0    1    -1   0
@@
 F 0 "L101" H 3830 4340 50  0000 L CNN
 F 1 "47 uH" H 3830 4260 50  0000 L CNN
-F 2 "" H 3800 4300 50  0001 C CNN
+F 2 "Capacitors_SMD:C_0805_HandSoldering" H 3800 4300 50  0001 C CNN
 F 3 "~" H 3800 4300 50  0001 C CNN
+F 4 "810-MLZ2012M470WT000" H 3800 4300 50  0001 C CNN "Mouser"
 	1    3800 4300
 	0    -1   -1   0
@@
 Wire Wire Line
 	3050 4550 3350 4550
-$Comp
-L Device:Q_PMOS_DSG Q103
-U 1 1 5C327542
-P 2650 4650
-F 0 "Q103" H 2850 4700 50  0000 L CNN
-F 1 "Q_PMOS_DSG" H 2850 4600 50  0000 L CNN
-F 2 "" H 2850 4750 50  0001 C CNN
-F 3 "~" H 2650 4650 50  0001 C CNN
-	1    2650 4650
-	0    1    -1   0
-$EndComp
 Wire Wire Line
 	2850 4550 3050 4550
@@
 $EndComp
 Wire Wire Line
-	2000 4550 2100 4550
-Wire Wire Line
 	2300 4550 2300 4700
 Wire Wire Line
@@
 L Connector_Generic:Conn_01x02 J101
 U 1 1 5C337705
-P 1100 4650
-F 0 "J101" H 1100 4750 50  0000 C CNN
-F 1 "Conn_01x02" H 1100 4450 50  0000 C CNN
-F 2 "" H 1100 4650 50  0001 C CNN
-F 3 "~" H 1100 4650 50  0001 C CNN
-	1    1100 4650
+P 1300 4650
+F 0 "J101" H 1300 4750 50  0000 C CNN
+F 1 "Conn_01x02" H 1300 4450 50  0000 C CNN
+F 2 "" H 1300 4650 50  0001 C CNN
+F 3 "~" H 1300 4650 50  0001 C CNN
+	1    1300 4650
 	-1   0    0    1
 $EndComp
@@
 L power:GND #PWR0152
 U 1 1 5C3377B2
-P 1400 4800
-F 0 "#PWR0152" H 1400 4550 50  0001 C CNN
-F 1 "GND" H 1400 4650 50  0000 C CNN
-F 2 "" H 1400 4800 50  0001 C CNN
-F 3 "" H 1400 4800 50  0001 C CNN
-	1    1400 4800
-	1    0    0    -1
-$EndComp
-Wire Wire Line
-	1400 4800 1400 4650
-Wire Wire Line
-	1400 4650 1300 4650
+P 1600 4800
+F 0 "#PWR0152" H 1600 4550 50  0001 C CNN
+F 1 "GND" H 1600 4650 50  0000 C CNN
+F 2 "" H 1600 4800 50  0001 C CNN
+F 3 "" H 1600 4800 50  0001 C CNN
+	1    1600 4800
+	1    0    0    -1
+$EndComp
+Wire Wire Line
+	1600 4800 1600 4650
+Wire Wire Line
+	1600 4650 1500 4650
 Wire Wire Line
 	2300 4900 2300 5050
@@
 	1950 6850 1950 6900
 $Comp
-L Device:Q_NPN_BEC Q?
+L Device:Q_NPN_BEC Q102
 U 1 1 5C66C411
 P 2200 5350
-F 0 "Q?" H 2400 5400 50  0000 L CNN
+F 0 "Q102" H 2400 5400 50  0000 L CNN
 F 1 "MMBT2222A-7-F" H 2400 5300 50  0000 L CNN
 F 2 "TO_SOT_Packages_SMD:SOT-23_Handsoldering" H 2400 5450 50  0001 C CNN
@@
 	1    0    0    -1
 $EndComp
+$Comp
+L Device:D_Schottky_Small D103
+U 1 1 5C0E0504
+P 1750 4550
+F 0 "D103" H 1700 4630 50  0000 L CNN
+F 1 "2SS100L-W" H 1470 4470 50  0000 L CNN
+F 2 "" V 1750 4550 50  0001 C CNN
+F 3 "~" V 1750 4550 50  0001 C CNN
+	1    1750 4550
+	-1   0    0    -1
+$EndComp
+Wire Wire Line
+	1650 4550 1500 4550
+$Comp
+L Device:Q_PMOS_GSD Q?
+U 1 1 5C140684
+P 2650 4650
+F 0 "Q?" H 2850 4700 50  0000 L CNN
+F 1 "BSS215PH6327XTSA1" H 2850 4600 50  0000 L CNN
+F 2 "TO_SOT_Packages_SMD:SOT-23_Handsoldering" H 2850 4750 50  0001 C CNN
+F 3 "~" H 2650 4650 50  0001 C CNN
+F 4 "726-BSS215PH6327" H 2650 4650 50  0001 C CNN "Mouser"
+	1    2650 4650
+	0    1    -1   0
+$EndComp
+Wire Wire Line
+	1850 4550 2100 4550
 $EndSCHEMATC

Commit message: Finish footprinting/sourcing all components
Parts:
- D101, D102, D103: footprint (none) -> receiver-footprints:Rectron_SOD-123FL; Mouser (none) -> 583-2SS100L-W
- J101: footprint (none) -> Socket_Strips:Socket_Strip_Straight_1x02_Pitch2.54mm; Mouser (none) -> NoPart
- gave numbers to parts that had none: 1
Changed lines of the file:
@@
 F 0 "D102" H 3450 6880 50  0000 L CNN
 F 1 "2SS100L-W" H 3220 6720 50  0000 L CNN
-F 2 "" V 3500 6800 50  0001 C CNN
+F 2 "receiver-footprints:Rectron_SOD-123FL" V 3500 6800 50  0001 C CNN
 F 3 "~" V 3500 6800 50  0001 C CNN
+F 4 "583-2SS100L-W" H 3500 6800 50  0001 C CNN "Mouser"
 	1    3500 6800
 	1    0    0    1
@@
 F 0 "D101" H 4350 4380 50  0000 L CNN
 F 1 "2SS100L-W" H 4120 4220 50  0000 L CNN
-F 2 "" V 4400 4300 50  0001 C CNN
+F 2 "receiver-footprints:Rectron_SOD-123FL" V 4400 4300 50  0001 C CNN
 F 3 "~" V 4400 4300 50  0001 C CNN
+F 4 "583-2SS100L-W" V 4400 4300 50  0001 C CNN "Mouser"
 	1    4400 4300
 	-1   0    0    -1
@@
 F 0 "J101" H 1300 4750 50  0000 C CNN
 F 1 "Conn_01x02" H 1300 4450 50  0000 C CNN
-F 2 "" H 1300 4650 50  0001 C CNN
+F 2 "Socket_Strips:Socket_Strip_Straight_1x02_Pitch2.54mm" H 1300 4650 50  0001 C CNN
 F 3 "~" H 1300 4650 50  0001 C CNN
+F 4 "NoPart" H 1300 4650 50  0001 C CNN "Mouser"
 	1    1300 4650
 	-1   0    0    1
@@
 F 0 "D103" H 1700 4630 50  0000 L CNN
 F 1 "2SS100L-W" H 1470 4470 50  0000 L CNN
-F 2 "" V 1750 4550 50  0001 C CNN
+F 2 "receiver-footprints:Rectron_SOD-123FL" V 1750 4550 50  0001 C CNN
 F 3 "~" V 1750 4550 50  0001 C CNN
+F 4 "583-2SS100L-W" V 1750 4550 50  0001 C CNN "Mouser"
 	1    1750 4550
 	-1   0    0    -1
@@
 	1650 4550 1500 4550
 $Comp
-L Device:Q_PMOS_GSD Q?
+L Device:Q_PMOS_GSD Q101
 U 1 1 5C140684
 P 2650 4650
-F 0 "Q?" H 2850 4700 50  0000 L CNN
+F 0 "Q101" H 2850 4700 50  0000 L CNN
 F 1 "BSS215PH6327XTSA1" H 2850 4600 50  0000 L CNN
 F 2 "TO_SOT_Packages_SMD:SOT-23_Handsoldering" H 2850 4750 50  0001 C CNN

Commit message: Most of the layout done TODO add test points for +12V, AVR_UART, various amplifier stage outputs
Connections:
- net -12V: now also C106.2, C109.2, C114.2, C116.2; no longer C106.1, C109.1, C114.1, C116.1
- net GND: now also C106.1, C109.1, C114.1, C116.1; no longer C106.2, C109.2, C114.2, C116.2
Changed lines of the file:
@@
 F 4 "647-UWX1E4R7MCL1" H 3750 7000 50  0001 C CNN "Mouser"
 	1    3750 7000
-	1    0    0    -1
+	1    0    0    1
 $EndComp
 $Comp
@@
 F 4 "647-UWX1E4R7MCL1" H 4150 7000 50  0001 C CNN "Mouser"
 	1    4150 7000
-	1    0    0    -1
+	1    0    0    1
 $EndComp
 $Comp
@@
 F 4 "647-UWX1E4R7MCL1" H 4500 7000 50  0001 C CNN "Mouser"
 	1    4500 7000
-	1    0    0    -1
+	1    0    0    1
 $EndComp
 $Comp
@@
 F 4 "647-UWX1E4R7MCL1" H 4850 7000 50  0001 C CNN "Mouser"
 	1    4850 7000
-	1    0    0    -1
+	1    0    0    1
 $EndComp
 $Comp

Commit message: Add copper fills and outline, autofill test point footprints, TODO finish placing test points and moving silkscreen
Parts:
- added TP101, TP102: TestPoint, Measurement_Points:Measurement_Point_Round-SMD-Pad_Small, symbol Connector:TestPoint
Connections:
- net +12V: now also TP102.1
- net -12V: now also TP101.1
Changed lines of the file:
@@
 Connection ~ 5750 4300
 Wire Wire Line
-	5750 4300 5400 4300
+	5750 4300 5550 4300
 Wire Wire Line
 	6100 4300 6100 4450
@@
 $EndComp
 Wire Wire Line
-	4950 6650 4950 6800
+	4950 6650 4950 6700
 Connection ~ 4950 6800
 Wire Wire Line
@@
 Wire Wire Line
 	1850 4550 2100 4550
+$Comp
+L Connector:TestPoint TP102
+U 1 1 5C2F2529
+P 5550 4150
+F 0 "TP102" H 5550 4420 50  0000 C CNN
+F 1 "TestPoint" H 5550 4350 50  0000 C CNN
+F 2 "Measurement_Points:Measurement_Point_Round-SMD-Pad_Small" H 5750 4150 50  0001 C CNN
+F 3 "~" H 5750 4150 50  0001 C CNN
+F 4 "NoPart" H 5750 4150 50  0001 C CNN "Mouser"
+	1    5550 4150
+	1    0    0    -1
+$EndComp
+Wire Wire Line
+	5550 4150 5550 4300
+Connection ~ 5550 4300
+Wire Wire Line
+	5550 4300 5400 4300
+$Comp
+L Connector:TestPoint TP101
+U 1 1 5C2F7F38
+P 5200 6700
+F 0 "TP101" H 5200 6970 50  0000 C CNN
+F 1 "TestPoint" H 5200 6900 50  0000 C CNN
+F 2 "Measurement_Points:Measurement_Point_Round-SMD-Pad_Small" H 5400 6700 50  0001 C CNN
+F 3 "~" H 5400 6700 50  0001 C CNN
+F 4 "NoPart" H 5200 6700 50  0001 C CNN "Mouser"
+	1    5200 6700
+	0    1    1    0
+$EndComp
+Wire Wire Line
+	5200 6700 4950 6700
+Connection ~ 4950 6700
+Wire Wire Line
+	4950 6700 4950 6800
 $EndSCHEMATC
