File: pcb/receiver/receiver.kicad_pcb (KiCad board)
At the start: 2 copper layers, 0 parts

Commit message: Most of the layout done TODO add test points for +12V, AVR_UART, various amplifier stage outputs
Parts:
- added C101: 10 uF, Capacitors_SMD:C_0805_HandSoldering, F.Cu at (86.0, 146.4)
- added C102: 4.7 nF, Capacitors_SMD:C_0402, F.Cu at (87.2, 154.0)
- added C103: 100 nF, Capacitors_SMD:C_0603_HandSoldering, F.Cu at (87.2, 150.9)
- added C104: 10 uF, Capacitors_SMD:C_0805_HandSoldering, F.Cu at (72.2, 129.2)
- added C105: 100 nF, Capacitors_SMD:C_0603_HandSoldering, F.Cu at (72.2, 131.1)
- added C106: 4.7 uF, Capacitors_SMD:CP_Elec_4x5.3, F.Cu at (71.2, 151.4)
- added C107: 1 nF, Capacitors_SMD:C_0402, F.Cu at (67.8, 140.9)
- added C108: 4.7 uF, Capacitors_SMD:CP_Elec_4x5.3, F.Cu at (79.8, 136.1)
- added C109: 4.7 uF, Capacitors_SMD:CP_Elec_4x5.3, F.Cu at (84.5, 188.0)
- added C110: 100 nF, Capacitors_SMD:C_0603_HandSoldering, F.Cu at (83.6, 155.4)
- added C111: 100 nF, Capacitors_SMD:C_0603_HandSoldering, F.Cu at (83.7, 157.3)
- added C112: 10 pF, Capacitors_SMD:C_0402, F.Cu at (80.0, 159.4)
- added C113: 4.7 uF, Capacitors_SMD:CP_Elec_4x5.3, F.Cu at (79.8, 143.3)
- added C114: 4.7 uF, Capacitors_SMD:CP_Elec_4x5.3, F.Cu at (86.3, 181.2)
- added C115: 10 uF, Capacitors_SMD:C_0805_HandSoldering, F.Cu at (76.2, 137.2)
- added C116: 4.7 uF, Capacitors_SMD:CP_Elec_4x5.3, F.Cu at (76.8, 151.4)
- added C117: 10 uF, Capacitors_SMD:C_0805_HandSoldering, F.Cu at (76.2, 142.3)
- added C201: 1 uF, Capacitors_SMD:C_0603_HandSoldering, F.Cu at (62.6, 185.0)
- added C202: 1 uF, Capacitors_SMD:C_0603_HandSoldering, F.Cu at (65.9, 179.1)
- added C203: 10 uF, Capacitors_SMD:C_0805_HandSoldering, B.Cu at (33.0, 186.1)
- added C204: 1 uF, Capacitors_SMD:C_0603_HandSoldering, F.Cu at (44.8, 189.0)
- added C205: 10 uF, Capacitors_SMD:C_0805_HandSoldering, B.Cu at (33.2, 180.0)
- added C206: 10 uF, Capacitors_SMD:C_0805_HandSoldering, F.Cu at (81.8, 182.0)
- added C207: 100 nF, Capacitors_SMD:C_0603_HandSoldering, F.Cu at (76.0, 185.0)
- added C208: 33 nF, Capacitors_SMD:C_0402, F.Cu at (34.8, 179.9)
- added C209: 1 uF, Capacitors_SMD:C_0603_HandSoldering, F.Cu at (76.0, 186.4)
- added C210: 2 pF, Capacitors_SMD:C_0603_HandSoldering, F.Cu at (38.2, 178.1)
- added C211: 10 uF, Capacitors_SMD:C_0805_HandSoldering, F.Cu at (35.1, 172.2)
- added C212: 100 nF, Capacitors_SMD:C_0603_HandSoldering, F.Cu at (42.1, 186.1)
- added C213: 1 nF, Capacitors_SMD:C_0402, F.Cu at (34.8, 175.8)
- added C214: 150 nF, Capacitors_SMD:C_0603_HandSoldering, F.Cu at (42.0, 177.9)
- added C215: 1 uF, Capacitors_SMD:C_0603_HandSoldering, F.Cu at (64.8, 175.4)
- added C216: 1 uF, Capacitors_SMD:C_0603_HandSoldering, F.Cu at (79.5, 174.2)
- added C217: 100 nF, Capacitors_SMD:C_0603_HandSoldering, F.Cu at (50.6, 177.9)
- added C218: 100 nF, Capacitors_SMD:C_0603_HandSoldering, F.Cu at (43.8, 186.1)
- added C219: 56 pF, Capacitors_SMD:C_0402, F.Cu at (48.8, 182.2)
- added C220: 100 nF, Capacitors_SMD:C_0603_HandSoldering, F.Cu at (76.6, 174.2)
- added C221: 1 uF, Capacitors_SMD:C_0603_HandSoldering, F.Cu at (59.9, 172.1)
- added C222: 10 uF, Capacitors_SMD:C_0805_HandSoldering, F.Cu at (58.9, 178.3)
- added C223: 3.3 nF, Capacitors_SMD:C_0603_HandSoldering, F.Cu at (49.9, 173.9)
- added C224: 33 nF, Capacitors_SMD:C_0402, F.Cu at (48.9, 171.6)
- added C225: 100 nF, Capacitors_SMD:C_0603_HandSoldering, F.Cu at (52.4, 168.2)
- added C226: 10 uF, Capacitors_SMD:C_0805_HandSoldering, F.Cu at (70.7, 170.1)
- added C227: 1 uF, Capacitors_SMD:C_0603_HandSoldering, B.Cu at (70.7, 174.3)
- added C228: 2 pF, Capacitors_SMD:C_0603_HandSoldering, F.Cu at (53.9, 162.7)
- added C229: 100 nF, Capacitors_SMD:C_0603_HandSoldering, F.Cu at (52.3, 149.2)
- added C230: 3.3 nF, Capacitors_SMD:C_0603_HandSoldering, F.Cu at (44.9, 166.9)
- added C231: 33 nF, Capacitors_SMD:C_0402, F.Cu at (44.9, 162.1)
- added C232: 10 pF DNP, Capacitors_SMD:C_0402, F.Cu at (43.9, 152.6)
- added C233: 270 pF, Capacitors_SMD:C_0402, F.Cu at (47.5, 152.6)
- added C234: 10 uF, Capacitors_SMD:C_0805_HandSoldering, F.Cu at (45.3, 178.0)
- added C235: 1 uF, Capacitors_SMD:C_0603_HandSoldering, B.Cu at (42.9, 182.1)
- added C236: 100 nF, Capacitors_SMD:C_0603_HandSoldering, F.Cu at (52.1, 156.1)
- added C237: 10 uF, Capacitors_SMD:C_0805_HandSoldering, F.Cu at (46.6, 162.1)
- added C238: 1 uF, Capacitors_SMD:C_0603_HandSoldering, B.Cu at (49.9, 162.7)
- added C239: 100 nF, Capacitors_SMD:C_0603_HandSoldering, F.Cu at (52.3, 184.7)
- added C240: 100 nF, Capacitors_SMD:C_0603_HandSoldering, F.Cu at (37.9, 164.7)
- added C241: 100 nF, Capacitors_SMD:C_0603_HandSoldering, F.Cu at (67.3, 185.0)
- added C242: 100 nF, Capacitors_SMD:C_0603_HandSoldering, F.Cu at (52.4, 186.6)
- added C243: 100 nF, Capacitors_SMD:C_0603_HandSoldering, F.Cu at (52.4, 188.6)
- added C244: 100 nF, Capacitors_SMD:C_0603_HandSoldering, F.Cu at (33.8, 163.0)
- added C245: 100 nF DNP, Capacitors_SMD:C_0603_HandSoldering, F.Cu at (33.8, 161.1)
- added C246: 100 nF, Capacitors_SMD:C_0603_HandSoldering, F.Cu at (76.0, 187.9)
- added C301: 1 uF, Capacitors_SMD:C_0603_HandSoldering, B.Cu at (51.0, 132.3)
- added C302: 100 nF, Capacitors_SMD:C_0603_HandSoldering, B.Cu at (51.0, 133.8)
- added C303: 100 nF, Capacitors_SMD:C_0603_HandSoldering, F.Cu at (41.7, 119.1)
- added C304: 100 nF, Capacitors_SMD:C_0603_HandSoldering, F.Cu at (75.2, 165.1)
- added C305: 100 nF, Capacitors_SMD:C_0603_HandSoldering, B.Cu at (51.0, 126.7)
- added C306: 100 nF, Capacitors_SMD:C_0603_HandSoldering, F.Cu at (52.3, 124.0)
- added C307: 100 nF, Capacitors_SMD:C_0603_HandSoldering, B.Cu at (51.0, 125.2)
- added C308: 100 nF, Capacitors_SMD:C_0603_HandSoldering, B.Cu at (47.1, 126.7)
- added C309: 100 nF, Capacitors_SMD:C_0603_HandSoldering, B.Cu at (47.2, 125.2)
- added C310: 4.7 uF, Capacitors_SMD:CP_Elec_4x5.3, F.Cu at (58.4, 123.8)
- added C311: 1 nF, Capacitors_SMD:C_0402, F.Cu at (38.2, 153.8)
- added C312: 100 nF, Capacitors_SMD:C_0603_HandSoldering, F.Cu at (36.2, 149.7)
- added C313: 100 pF, Capacitors_SMD:C_0402, F.Cu at (31.6, 144.8)
- added C314: 10 uF, Capacitors_SMD:C_0805_HandSoldering, B.Cu at (34.4, 140.1)
- added C315: 10 uF, Capacitors_SMD:C_0805_HandSoldering, B.Cu at (36.5, 140.1)
- added C316: 100 nF, Capacitors_SMD:C_0603_HandSoldering, F.Cu at (38.3, 141.0)
- added C317: 100 nF, Capacitors_SMD:C_0603_HandSoldering, F.Cu at (38.3, 142.5)
- added C318: 100 nF, Capacitors_SMD:C_0603_HandSoldering, F.Cu at (34.4, 132.6)
- added C319: 10 uF, Capacitors_SMD:C_0805_HandSoldering, B.Cu at (34.4, 132.6)
- added C320: 100 nF, Capacitors_SMD:C_0603_HandSoldering, F.Cu at (62.2, 121.9)
- added C321: 100 nF, Capacitors_SMD:C_0603_HandSoldering, F.Cu at (71.1, 122.1)
- added C322: 22 pF, Capacitors_SMD:C_0402, F.Cu at (47.8, 136.6)
- added C323: 22 pF, Capacitors_SMD:C_0402, F.Cu at (50.0, 136.6)
- added D101: 2SS100L-W, receiver-footprints:Rectron_SOD-123FL, F.Cu at (72.0, 140.9)
- added D102: 2SS100L-W, receiver-footprints:Rectron_SOD-123FL, F.Cu at (80.5, 151.6)
- added D103: 2SS100L-W, receiver-footprints:Rectron_SOD-123FL, F.Cu at (79.7, 122.5)
- added D201: QSB34CGR, receiver-footprints:Fairchild_QSB34CGR, F.Cu at (36.8, 186.0)
- added D202: BPW 34 S-Z, receiver-footprints:OSRAM_BPW34S-Z, F.Cu at (36.8, 186.0)
- added D203: TEFD4300F, LEDs:LED_D3.0mm, F.Cu at (36.8, 184.7)
- added D205: PLZ4V7B-G3/H, receiver-footprints:Vishay_DO-219AC, F.Cu at (43.5, 156.8)
- added D301: 2SS100L-W, receiver-footprints:Rectron_SOD-123FL, F.Cu at (66.8, 117.1)
- added D302: 2SS100L-W, receiver-footprints:Rectron_SOD-123FL, F.Cu at (36.3, 147.2)
- added D303: 2SS100L-W, receiver-footprints:Rectron_SOD-123FL, F.Cu at (31.6, 147.2)
- added D304: TPD1E04U04DPYR, receiver-footprints:TI_X1SON, F.Cu at (51.6, 120.3)
- added D305: TPD1E04U04DPYR, receiver-footprints:TI_X1SON, F.Cu at (48.8, 122.2)
- added D306: TPD1E04U04DPYR, receiver-footprints:TI_X1SON, F.Cu at (51.0, 122.2)
- added J101: Conn_01x02, Socket_Strips:Socket_Strip_Straight_1x02_Pitch2.54mm, F.Cu at (77.2, 117.2)
- added J301: UART, Socket_Strips:Socket_Strip_Straight_1x03_Pitch2.54mm, F.Cu at (61.1, 148.0)
- added J302: STM32_SWD, Socket_Strips:Socket_Strip_Straight_2x02_Pitch2.54mm, F.Cu at (42.8, 123.2)
- added J303: AVR_DEBUG, Socket_Strips:Socket_Strip_Straight_1x03_Pitch2.54mm, F.Cu at (86.5, 162.7)
- added J304: USB_B_Micro, receiver-footprints:Amphenol_10118194, F.Cu at (49.4, 118.3)
- added L101: 47 uH, Capacitors_SMD:C_0805_HandSoldering, F.Cu at (72.0, 138.2)
- added L102: 10 uH, Capacitors_SMD:C_0805_HandSoldering, F.Cu at (82.5, 148.0)
- added Q101: BSS215PH6327XTSA1, TO_SOT_Packages_SMD:SOT-23_Handsoldering, F.Cu at (84.5, 128.8)
- added Q102: MMBT2222A-7-F, TO_SOT_Packages_SMD:SOT-23_Handsoldering, F.Cu at (79.7, 128.8)
- added Q201: BFR31,215, TO_SOT_Packages_SMD:SOT-23_Handsoldering, F.Cu at (31.3, 185.8)
- added Q202: MMBT2222A-7-F, TO_SOT_Packages_SMD:SOT-23_Handsoldering, F.Cu at (76.1, 182.0)
- added Q203: MMBT2222A-7-F, TO_SOT_Packages_SMD:SOT-23_Handsoldering, F.Cu at (31.3, 179.9)
- added Q204: MMBT2222A-7-F, TO_SOT_Packages_SMD:SOT-23_Handsoldering, F.Cu at (31.2, 173.9)
- added Q205: MMBT2222A-7-F, TO_SOT_Packages_SMD:SOT-23_Handsoldering, F.Cu at (58.9, 175.3)
- added Q206: MMBT2222A-7-F, TO_SOT_Packages_SMD:SOT-23_Handsoldering, F.Cu at (64.2, 159.0)
- added Q207: TF414T5G, receiver-footprints:ON_XDFN3, F.Cu at (56.3, 162.7)
- added R101: 10, Capacitors_SMD:C_0402, F.Cu at (87.7, 146.3)
- added R102: 680k, Resistors_SMD:R_0603_HandSoldering, F.Cu at (67.8, 137.5)
- added R103: 47k, Resistors_SMD:R_0603_HandSoldering, F.Cu at (67.8, 133.2)
- added R104: 120k, Resistors_SMD:R_0603_HandSoldering, F.Cu at (83.6, 159.2)
- added R105: 1.2M, Resistors_SMD:R_0402, F.Cu at (80.0, 158.1)
- added R106: 100k, Resistors_SMD:R_0402, F.Cu at (80.0, 156.8)
- added R107: 1k, Resistors_SMD:R_0603_HandSoldering, F.Cu at (72.1, 126.8)
- added R108: 100k, Resistors_SMD:R_0402, F.Cu at (84.5, 125.2)
- added R201: 100k, Resistors_SMD:R_0402, F.Cu at (70.6, 183.2)
- added R202: 10k, Resistors_SMD:R_0603_HandSoldering, F.Cu at (67.3, 182.0)
- added R203: 33, Resistors_SMD:R_0603_HandSoldering, F.Cu at (31.3, 189.4)
- added R204: 0, Resistors_SMD:R_0603_HandSoldering, F.Cu at (40.3, 190.7)
- added R205: 1k, Resistors_SMD:R_0603_HandSoldering, F.Cu at (44.7, 190.7)
- added R206: 10k, Resistors_SMD:R_0603_HandSoldering, F.Cu at (37.9, 163.0)
- added R207: 4k7, Resistors_SMD:R_0603_HandSoldering, F.Cu at (74.9, 178.8)
- added R208: 4k7, Resistors_SMD:R_0603_HandSoldering, F.Cu at (79.2, 178.8)
- added R209: 33, Resistors_SMD:R_0603_HandSoldering, B.Cu at (32.6, 176.7)
- added R210: 100k, Resistors_SMD:R_0402, F.Cu at (45.8, 185.8)
- added R211: 1M, Resistors_SMD:R_0603_HandSoldering, F.Cu at (38.2, 179.7)
- added R212: 100k, Resistors_SMD:R_0402, F.Cu at (34.8, 177.8)
- added R213: 100k DNP, Resistors_SMD:R_0402, F.Cu at (45.8, 186.9)
- added R214: 33, Resistors_SMD:R_0603_HandSoldering, B.Cu at (32.6, 172.5)
- added R215: 1M, Resistors_SMD:R_0603_HandSoldering, F.Cu at (31.4, 169.7)
- added R216: 4k7, Resistors_SMD:R_0603_HandSoldering, F.Cu at (38.4, 176.5)
- added R217: 10k, Resistors_SMD:R_0603_HandSoldering, F.Cu at (63.1, 175.4)
- added R218: 2k, Resistors_SMD:R_0603_HandSoldering, F.Cu at (43.6, 177.9)
- added R219: 100k, Resistors_SMD:R_0402, F.Cu at (45.8, 184.8)
- added R220: 10k, Resistors_SMD:R_0603_HandSoldering, F.Cu at (81.6, 174.2)
- added R221: 100k, Resistors_SMD:R_0402, F.Cu at (78.1, 174.2)
- added R222: 100k, Resistors_SMD:R_0402, F.Cu at (47.6, 182.2)
- added R223: 33, Resistors_SMD:R_0603_HandSoldering, F.Cu at (70.7, 178.1)
- added R224: 1k, Resistors_SMD:R_0603_HandSoldering, F.Cu at (49.0, 177.9)
- added R225: 12k DNP, Resistors_SMD:R_0603_HandSoldering, F.Cu at (59.8, 159.5)
- added R226: 12k, Resistors_SMD:R_0603_HandSoldering, F.Cu at (59.8, 157.0)
- added R227: 33, Resistors_SMD:R_0603_HandSoldering, F.Cu at (70.8, 168.2)
- added R228: 10k, Resistors_SMD:R_0603_HandSoldering, F.Cu at (48.9, 168.3)
- added R229: 10k, Resistors_SMD:R_0603_HandSoldering, F.Cu at (50.7, 168.3)
- added R230: 18k, Resistors_SMD:R_0603_HandSoldering, F.Cu at (64.0, 162.6)
- added R231: 470k, Resistors_SMD:R_0603_HandSoldering, F.Cu at (59.7, 162.6)
- added R232: 470k, Resistors_SMD:R_0603_HandSoldering, F.Cu at (55.0, 159.5)
- added R233: 1k, Resistors_SMD:R_0603_HandSoldering, F.Cu at (44.8, 165.1)
- added R234: 330k, Resistors_SMD:R_0402, F.Cu at (45.0, 152.6)
- added R235: 20k, Resistors_SMD:R_0402, F.Cu at (46.4, 152.6)
- added R236: 33, Resistors_SMD:R_0603_HandSoldering, F.Cu at (47.1, 178.0)
- added R237: 10k, Resistors_SMD:R_0603_HandSoldering, F.Cu at (47.6, 156.0)
- added R238: 10k, Resistors_SMD:R_0603_HandSoldering, F.Cu at (52.1, 157.7)
- added R239: 33, Resistors_SMD:R_0603_HandSoldering, B.Cu at (48.1, 162.7)
- added R240: 10k, Resistors_SMD:R_0603_HandSoldering, F.Cu at (38.0, 161.1)
- added R241: 10k, Resistors_SMD:R_0603_HandSoldering, F.Cu at (37.8, 159.4)
- added R242: 10k, Resistors_SMD:R_0603_HandSoldering, F.Cu at (37.9, 157.6)
- added R243: 51k, Resistors_SMD:R_0402, F.Cu at (48.7, 185.2)
- added R244: 30k, Resistors_SMD:R_0402, F.Cu at (48.7, 187.0)
- added R245: 20k, Resistors_SMD:R_0402, F.Cu at (48.7, 188.9)
- added R246: 1k DNP, Resistors_SMD:R_0603_HandSoldering, F.Cu at (79.9, 181.9)
- added R247: 10k DNP, Resistors_SMD:R_0603_HandSoldering, F.Cu at (70.7, 179.7)
- added R248: 4k7, Resistors_SMD:R_0603_HandSoldering, F.Cu at (47.6, 157.8)
- added R302: 0, Resistors_SMD:R_0603_HandSoldering, F.Cu at (61.4, 132.2)
- added R303: 0, Resistors_SMD:R_0603_HandSoldering, F.Cu at (61.2, 137.4)
- added R304: 0, Resistors_SMD:R_0603_HandSoldering, F.Cu at (61.3, 134.1)
- added R305: 0, Resistors_SMD:R_0603_HandSoldering, F.Cu at (61.3, 135.7)
- added R306: 1M, Resistors_SMD:R_0603_HandSoldering, F.Cu at (36.1, 151.4)
- added R307: 1M, Resistors_SMD:R_0603_HandSoldering, F.Cu at (31.8, 151.4)
- added R308: 47k, Resistors_SMD:R_0603_HandSoldering, F.Cu at (31.8, 149.7)
- added R309: 33, Resistors_SMD:R_0603_HandSoldering, F.Cu at (39.0, 137.6)
- added R310: 10k, Resistors_SMD:R_0603_HandSoldering, F.Cu at (36.1, 144.5)
- added R311: 100k DNP, Resistors_SMD:R_0402, B.Cu at (52.0, 128.3)
- added R312: 100k, Resistors_SMD:R_0402, F.Cu at (35.8, 132.6)
- added R313: 100k, Resistors_SMD:R_0402, F.Cu at (37.4, 136.4)
- added R314: 330, Resistors_SMD:R_0402, F.Cu at (58.1, 145.6)
- added R315: 330, Resistors_SMD:R_0402, F.Cu at (58.1, 143.2)
- added R316: 330, Resistors_SMD:R_0402, F.Cu at (84.0, 165.2)
- added R317: 10k, Resistors_SMD:R_0603_HandSoldering, F.Cu at (43.4, 135.3)
- added R318: 10k DNP, Resistors_SMD:R_0603_HandSoldering, F.Cu at (45.3, 135.3)
- added U101: TPS63700DRCR, receiver-footprints:TI-VSON10, F.Cu at (84.2, 151.8)
- added U102: NCP1403SNT1G, receiver-footprints:ON-TSOP-5, F.Cu at (72.1, 134.9)
- added U201: ADR550ARTZ-REEL7, TO_SOT_Packages_SMD:SOT-23_Handsoldering, F.Cu at (62.3, 182.0)
- added U202: TL974IPWR, receiver-footprints:TI-SOIC14, F.Cu at (70.7, 174.2)
- added U203: MAX4477AUA+, receiver-footprints:Maxim-uMAX8, F.Cu at (42.9, 182.1)
- added U204: OPA2141AIDR, receiver-footprints:TI-SOIC8, F.Cu at (49.9, 162.6)
- added U205: NLAS4599DFT2G, receiver-footprints:On-SOT363, F.Cu at (48.4, 149.5)
- added U301: ATTINY412-SSNR, receiver-footprints:Atmel-SOIC150-8, F.Cu at (79.2, 165.2)
- added U302: STM32F070F6P6, receiver-footprints:ST-TSSOP20, F.Cu at (51.0, 129.7)
- added U303: MAX11666AUB+T, receiver-footprints:Maxim-U10E+3, F.Cu at (34.4, 138.8)
- added U304: L78L33ABUTR, TO_SOT_Packages_SMD:SOT-89-3_Handsoldering, F.Cu at (66.6, 122.8)
- added Y301: ABM3B-8.000MHZ-10-1UT, Crystals:Crystal_SMD_Abracon_ABM3C-4pin_5.0x3.2mm, F.Cu at (48.5, 140.2)
Routing:
- net GND: track 0.00 -> 827.8 mm, vias 0 -> 72
- net /Digital/+3V3: track 0.00 -> 163.0 mm, vias 0 -> 12
- net +12V: track 0.00 -> 123.9 mm, vias 0 -> 6
- net /Photodiode/+10V: track 0.00 -> 104.7 mm, vias 0 -> 3
- net +5V_USB: track 0.00 -> 99.9 mm, vias 0 -> 4
- net -12V: track 0.00 -> 93.0 mm, vias 0 -> 2
- net /Digital/ATTINY_TXD: track 0.00 -> 51.4 mm
- net /Photodiode/+2V5: track 0.00 -> 42.3 mm, vias 0 -> 6
- net /Digital/ATTINY_RXD: track 0.00 -> 39.7 mm
- net /Photodiode/+5V0_PWR: track 0.00 -> 37.8 mm, vias 0 -> 2
- net /Digital/GAIN_SEL: track 0.00 -> 36.9 mm
- net /Digital/ADC_NSS: track 0.00 -> 35.1 mm, vias 0 -> 2
- net /Digital/GAIN_ADC: track 0.00 -> 34.8 mm, vias 0 -> 3
- net /Digital/ADC_SCK: track 0.00 -> 31.2 mm, vias 0 -> 2
- net Net-(C228-Pad1): track 0.00 -> 29.4 mm
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