File: pcb/receiver/digital.sch (KiCad schematic (older format))
At the start: 56 parts, among them J301 Conn_01x03, J302 Conn_01x04, J303 Conn_01x03, J304 USB_B_Micro, U301 ATTINY412-SSNR, U302 STM32F070F6P6, U303 MAX11666AUB+T, U304 L78L33ABUTR, Y301 ABM3B-8.000MHZ-10-1UT

Commit message: Autofill components
Parts:
- C301: footprint (none) -> Capacitors_SMD:C_0603_HandSoldering; Mouser (none) -> 710-885012106022
- C302, C303, C304, C305, C306, C307, C308, C309, C312, C316, C317, C318, C320, C321: footprint (none) -> Capacitors_SMD:C_0603_HandSoldering; Mouser (none) -> 710-885012206071
- C310: footprint (none) -> Capacitors_SMD:CP_Elec_4x5.3; Mouser (none) -> 647-UWX1E4R7MCL1
- C311: footprint (none) -> Capacitors_SMD:C_0402; Mouser (none) -> 710-885012205061
- C314, C315, C319: footprint (none) -> Capacitors_SMD:C_0805_HandSoldering; Mouser (none) -> 81-GRM21BR61E106MA3L
- C323: footprint (none) -> Capacitors_SMD:C_0402; Mouser (none) -> 710-885012005009
- R303, R304: footprint (none) -> Resistors_SMD:R_0603_HandSoldering; Mouser (none) -> 755-SFR03EZPJ000
- R306, R307: footprint (none) -> Resistors_SMD:R_0603_HandSoldering; Mouser (none) -> 603-RC0603JR-071ML
- R308: footprint (none) -> Resistors_SMD:R_0603_HandSoldering; Mouser (none) -> 603-RC0603FR-0747KL
- R309: footprint (none) -> Resistors_SMD:R_0603_HandSoldering; Mouser (none) -> 755-ESR03EZPJ330
- R310, R317: footprint (none) -> Resistors_SMD:R_0603_HandSoldering; Mouser (none) -> 603-RC0603FR-0710KL
- R312, R313: footprint (none) -> Resistors_SMD:R_0402; Mouser (none) -> 603-RC0402JR-13100KL
Changed lines of the file:
@@
 F 0 "C304" H 4760 5570 50  0000 L CNN
 F 1 "100 nF" H 4760 5420 50  0000 L CNN
-F 2 "" H 4750 5500 50  0001 C CNN
+F 2 "Capacitors_SMD:C_0603_HandSoldering" H 4750 5500 50  0001 C CNN
 F 3 "~" H 4750 5500 50  0001 C CNN
+F 4 "710-885012206071" H 4750 5500 50  0001 C CNN "Mouser"
 	1    4750 5500
 	1    0    0    1
@@
 F 0 "C305" H 9360 1870 50  0000 L CNN
 F 1 "100 nF" H 9360 1720 50  0000 L CNN
-F 2 "" H 9350 1800 50  0001 C CNN
+F 2 "Capacitors_SMD:C_0603_HandSoldering" H 9350 1800 50  0001 C CNN
 F 3 "~" H 9350 1800 50  0001 C CNN
+F 4 "710-885012206071" H 9350 1800 50  0001 C CNN "Mouser"
 	1    9350 1800
 	1    0    0    -1
@@
 F 0 "C306" H 9710 1870 50  0000 L CNN
 F 1 "100 nF" H 9710 1720 50  0000 L CNN
-F 2 "" H 9700 1800 50  0001 C CNN
+F 2 "Capacitors_SMD:C_0603_HandSoldering" H 9700 1800 50  0001 C CNN
 F 3 "~" H 9700 1800 50  0001 C CNN
+F 4 "710-885012206071" H 9700 1800 50  0001 C CNN "Mouser"
 	1    9700 1800
 	1    0    0    -1
@@
 F 0 "C307" H 10010 1870 50  0000 L CNN
 F 1 "100 nF" H 10010 1720 50  0000 L CNN
-F 2 "" H 10000 1800 50  0001 C CNN
+F 2 "Capacitors_SMD:C_0603_HandSoldering" H 10000 1800 50  0001 C CNN
 F 3 "~" H 10000 1800 50  0001 C CNN
+F 4 "710-885012206071" H 10000 1800 50  0001 C CNN "Mouser"
 	1    10000 1800
 	1    0    0    -1
@@
 F 0 "C308" H 10310 1870 50  0000 L CNN
 F 1 "100 nF" H 10310 1720 50  0000 L CNN
-F 2 "" H 10300 1800 50  0001 C CNN
+F 2 "Capacitors_SMD:C_0603_HandSoldering" H 10300 1800 50  0001 C CNN
 F 3 "~" H 10300 1800 50  0001 C CNN
+F 4 "710-885012206071" H 10300 1800 50  0001 C CNN "Mouser"
 	1    10300 1800
 	1    0    0    -1
@@
 F 0 "C309" H 10610 1870 50  0000 L CNN
 F 1 "100 nF" H 10610 1720 50  0000 L CNN
-F 2 "" H 10600 1800 50  0001 C CNN
+F 2 "Capacitors_SMD:C_0603_HandSoldering" H 10600 1800 50  0001 C CNN
 F 3 "~" H 10600 1800 50  0001 C CNN
+F 4 "710-885012206071" H 10600 1800 50  0001 C CNN "Mouser"
 	1    10600 1800
 	1    0    0    -1
@@
 F 0 "C310" H 10910 1870 50  0000 L CNN
 F 1 "4.7 uF" H 10910 1720 50  0000 L CNN
-F 2 "" H 10900 1800 50  0001 C CNN
+F 2 "Capacitors_SMD:CP_Elec_4x5.3" H 10900 1800 50  0001 C CNN
 F 3 "~" H 10900 1800 50  0001 C CNN
+F 4 "647-UWX1E4R7MCL1" H 10900 1800 50  0001 C CNN "Mouser"
 	1    10900 1800
 	1    0    0    -1
@@
 F 0 "C303" H 1910 1570 50  0000 L CNN
 F 1 "100 nF" H 1910 1420 50  0000 L CNN
-F 2 "" H 1900 1500 50  0001 C CNN
+F 2 "Capacitors_SMD:C_0603_HandSoldering" H 1900 1500 50  0001 C CNN
 F 3 "~" H 1900 1500 50  0001 C CNN
+F 4 "710-885012206071" H 1900 1500 50  0001 C CNN "Mouser"
 	1    1900 1500
 	0    1    -1   0
@@
 F 0 "C302" H 1760 1920 50  0000 L CNN
 F 1 "100 nF" H 1760 1770 50  0000 L CNN
-F 2 "" H 1750 1850 50  0001 C CNN
+F 2 "Capacitors_SMD:C_0603_HandSoldering" H 1750 1850 50  0001 C CNN
 F 3 "~" H 1750 1850 50  0001 C CNN
+F 4 "710-885012206071" H 1750 1850 50  0001 C CNN "Mouser"
 	1    1750 1850
 	1    0    0    -1
@@
 F 0 "C301" H 1510 1920 50  0000 L CNN
 F 1 "1 uF" H 1510 1770 50  0000 L CNN
-F 2 "" H 1500 1850 50  0001 C CNN
+F 2 "Capacitors_SMD:C_0603_HandSoldering" H 1500 1850 50  0001 C CNN
 F 3 "~" H 1500 1850 50  0001 C CNN
+F 4 "710-885012106022" H 1500 1850 50  0001 C CNN "Mouser"
 	1    1500 1850
 	1    0    0    -1
@@
 F 0 "R303" H 1980 3270 50  0000 L CNN
 F 1 "0" H 1980 3210 50  0000 L CNN
-F 2 "" H 1950 3250 50  0001 C CNN
+F 2 "Resistors_SMD:R_0603_HandSoldering" H 1950 3250 50  0001 C CNN
 F 3 "~" H 1950 3250 50  0001 C CNN
+F 4 "755-SFR03EZPJ000" H 1950 3250 50  0001 C CNN "Mouser"
 	1    1950 3250
 	0    -1   -1   0
@@
 F 0 "R304" H 1980 3370 50  0000 L CNN
 F 1 "0" H 1980 3310 50  0000 L CNN
-F 2 "" H 1950 3350 50  0001 C CNN
+F 2 "Resistors_SMD:R_0603_HandSoldering" H 1950 3350 50  0001 C CNN
 F 3 "~" H 1950 3350 50  0001 C CNN
+F 4 "755-SFR03EZPJ000" H 1950 3350 50  0001 C CNN "Mouser"
 	1    1950 3350
 	0    -1   1    0
@@
 F 0 "R309" H 5880 3720 50  0000 L CNN
 F 1 "33" H 5880 3660 50  0000 L CNN
-F 2 "" H 5850 3700 50  0001 C CNN
+F 2 "Resistors_SMD:R_0603_HandSoldering" H 5850 3700 50  0001 C CNN
 F 3 "~" H 5850 3700 50  0001 C CNN
+F 4 "755-ESR03EZPJ330" H 5850 3700 50  0001 C CNN "Mouser"
 	1    5850 3700
 	0    -1   1    0
@@
 F 0 "C315" H 6460 4420 50  0000 L CNN
 F 1 "10 uF" H 6460 4270 50  0000 L CNN
-F 2 "" H 6450 4350 50  0001 C CNN
+F 2 "Capacitors_SMD:C_0805_HandSoldering" H 6450 4350 50  0001 C CNN
 F 3 "~" H 6450 4350 50  0001 C CNN
+F 4 "81-GRM21BR61E106MA3L" H 6450 4350 50  0001 C CNN "Mouser"
 	1    6450 4350
 	-1   0    0    -1
@@
 F 0 "C314" H 6110 4420 50  0000 L CNN
 F 1 "10 uF" H 6110 4270 50  0000 L CNN
-F 2 "" H 6100 4350 50  0001 C CNN
+F 2 "Capacitors_SMD:C_0805_HandSoldering" H 6100 4350 50  0001 C CNN
 F 3 "~" H 6100 4350 50  0001 C CNN
+F 4 "81-GRM21BR61E106MA3L" H 6100 4350 50  0001 C CNN "Mouser"
 	1    6100 4350
 	-1   0    0    -1
@@
 F 0 "C316" H 6760 4420 50  0000 L CNN
 F 1 "100 nF" H 6760 4270 50  0000 L CNN
-F 2 "" H 6750 4350 50  0001 C CNN
+F 2 "Capacitors_SMD:C_0603_HandSoldering" H 6750 4350 50  0001 C CNN
 F 3 "~" H 6750 4350 50  0001 C CNN
+F 4 "710-885012206071" H 6750 4350 50  0001 C CNN "Mouser"
 	1    6750 4350
 	-1   0    0    -1
@@
 F 0 "C317" H 7060 4420 50  0000 L CNN
 F 1 "100 nF" H 7060 4270 50  0000 L CNN
-F 2 "" H 7050 4350 50  0001 C CNN
+F 2 "Capacitors_SMD:C_0603_HandSoldering" H 7050 4350 50  0001 C CNN
 F 3 "~" H 7050 4350 50  0001 C CNN
+F 4 "710-885012206071" H 7050 4350 50  0001 C CNN "Mouser"
 	1    7050 4350
 	-1   0    0    -1
@@
 F 0 "R312" H 8080 3920 50  0000 L CNN
 F 1 "100k" H 8080 3860 50  0000 L CNN
-F 2 "" H 8050 3900 50  0001 C CNN
+F 2 "Resistors_SMD:R_0402" H 8050 3900 50  0001 C CNN
 F 3 "~" H 8050 3900 50  0001 C CNN
+F 4 "603-RC0402JR-13100KL" H 8050 3900 50  0001 C CNN "Mouser"
 	1    8050 3900
 	1    0    0    -1
@@
 F 0 "C318" H 8010 3370 50  0000 L CNN
 F 1 "100 nF" H 8010 3220 50  0000 L CNN
-F 2 "" H 8000 3300 50  0001 C CNN
+F 2 "Capacitors_SMD:C_0603_HandSoldering" H 8000 3300 50  0001 C CNN
 F 3 "~" H 8000 3300 50  0001 C CNN
+F 4 "710-885012206071" H 8000 3300 50  0001 C CNN "Mouser"
 	1    8000 3300
 	1    0    0    1
@@
 F 0 "C319" H 8360 3370 50  0000 L CNN
 F 1 "10 uF" H 8360 3220 50  0000 L CNN
-F 2 "" H 8350 3300 50  0001 C CNN
+F 2 "Capacitors_SMD:C_0805_HandSoldering" H 8350 3300 50  0001 C CNN
 F 3 "~" H 8350 3300 50  0001 C CNN
+F 4 "81-GRM21BR61E106MA3L" H 8350 3300 50  0001 C CNN "Mouser"
 	1    8350 3300
 	1    0    0    1
@@
 F 0 "R310" H 6230 3420 50  0000 L CNN
 F 1 "10k" H 6230 3360 50  0000 L CNN
-F 2 "" H 6200 3400 50  0001 C CNN
+F 2 "Resistors_SMD:R_0603_HandSoldering" H 6200 3400 50  0001 C CNN
 F 3 "~" H 6200 3400 50  0001 C CNN
+F 4 "603-RC0603FR-0710KL" H 6200 3400 50  0001 C CNN "Mouser"
 	1    6200 3400
 	0    -1   -1   0
@@
 F 0 "C311" H 3660 3370 50  0000 L CNN
 F 1 "1 nF" H 3660 3220 50  0000 L CNN
-F 2 "" H 3650 3300 50  0001 C CNN
+F 2 "Capacitors_SMD:C_0402" H 3650 3300 50  0001 C CNN
 F 3 "~" H 3650 3300 50  0001 C CNN
+F 4 "710-885012205061" H 3650 3300 50  0001 C CNN "Mouser"
 	1    3650 3300
 	0    -1   -1   0
@@
 F 0 "R307" H 3880 3520 50  0000 L CNN
 F 1 "1M" H 3880 3460 50  0000 L CNN
-F 2 "" H 3850 3500 50  0001 C CNN
+F 2 "Resistors_SMD:R_0603_HandSoldering" H 3850 3500 50  0001 C CNN
 F 3 "~" H 3850 3500 50  0001 C CNN
+F 4 "603-RC0603JR-071ML" H 3850 3500 50  0001 C CNN "Mouser"
 	1    3850 3500
 	1    0    0    -1
@@
 F 0 "R306" H 3880 3120 50  0000 L CNN
 F 1 "1M" H 3880 3060 50  0000 L CNN
-F 2 "" H 3850 3100 50  0001 C CNN
+F 2 "Resistors_SMD:R_0603_HandSoldering" H 3850 3100 50  0001 C CNN
 F 3 "~" H 3850 3100 50  0001 C CNN
+F 4 "603-RC0603JR-071ML" H 3850 3100 50  0001 C CNN "Mouser"
 	1    3850 3100
 	1    0    0    -1
@@
 F 0 "R308" H 4230 3320 50  0000 L CNN
 F 1 "47k" H 4230 3260 50  0000 L CNN
-F 2 "" H 4200 3300 50  0001 C CNN
+F 2 "Resistors_SMD:R_0603_HandSoldering" H 4200 3300 50  0001 C CNN
 F 3 "~" H 4200 3300 50  0001 C CNN
+F 4 "603-RC0603FR-0747KL" H 4200 3300 50  0001 C CNN "Mouser"
 	1    4200 3300
 	0    -1   1    0
@@
 F 0 "C312" H 4060 2970 50  0000 L CNN
 F 1 "100 nF" H 4060 2820 50  0000 L CNN
-F 2 "" H 4050 2900 50  0001 C CNN
+F 2 "Capacitors_SMD:C_0603_HandSoldering" H 4050 2900 50  0001 C CNN
 F 3 "~" H 4050 2900 50  0001 C CNN
+F 4 "710-885012206071" H 4050 2900 50  0001 C CNN "Mouser"
 	1    4050 2900
 	0    -1   -1   0
@@
 F 0 "R313" H 8280 3720 50  0000 L CNN
 F 1 "100k" H 8280 3660 50  0000 L CNN
-F 2 "" H 8250 3700 50  0001 C CNN
+F 2 "Resistors_SMD:R_0402" H 8250 3700 50  0001 C CNN
 F 3 "~" H 8250 3700 50  0001 C CNN
+F 4 "603-RC0402JR-13100KL" H 8250 3700 50  0001 C CNN "Mouser"
 	1    8250 3700
 	0    -1   1    0
@@
 F 0 "C320" H 1560 6020 50  0000 L CNN
 F 1 "100 nF" H 1560 5870 50  0000 L CNN
-F 2 "" H 1550 5950 50  0001 C CNN
+F 2 "Capacitors_SMD:C_0603_HandSoldering" H 1550 5950 50  0001 C CNN
 F 3 "~" H 1550 5950 50  0001 C CNN
+F 4 "710-885012206071" H 1550 5950 50  0001 C CNN "Mouser"
 	1    1550 5950
 	1    0    0    -1
@@
 F 0 "C321" H 2860 6020 50  0000 L CNN
 F 1 "100 nF" H 2860 5870 50  0000 L CNN
-F 2 "" H 2850 5950 50  0001 C CNN
+F 2 "Capacitors_SMD:C_0603_HandSoldering" H 2850 5950 50  0001 C CNN
 F 3 "~" H 2850 5950 50  0001 C CNN
+F 4 "710-885012206071" H 2850 5950 50  0001 C CNN "Mouser"
 	1    2850 5950
 	1    0    0    -1
@@
 F 0 "C323" H 1310 1920 50  0000 L CNN
 F 1 "22 pF" H 1310 1770 50  0000 L CNN
-F 2 "" H 1300 1850 50  0001 C CNN
+F 2 "Capacitors_SMD:C_0402" H 1300 1850 50  0001 C CNN
 F 3 "~" H 1300 1850 50  0001 C CNN
+F 4 "710-885012005009" H 1300 1850 50  0001 C CNN "Mouser"
 	1    1300 1850
 	-1   0    0    -1
@@
 F 0 "R317" H 2380 720 50  0000 L CNN
 F 1 "10k" H 2380 660 50  0000 L CNN
-F 2 "" H 2350 700 50  0001 C CNN
+F 2 "Resistors_SMD:R_0603_HandSoldering" H 2350 700 50  0001 C CNN
 F 3 "~" H 2350 700 50  0001 C CNN
+F 4 "603-RC0603FR-0710KL" H 2350 700 50  0001 C CNN "Mouser"
 	1    2350 700
 	0    -1   1    0

Commit message: Footprint more stuff
Parts:
- removed D301: D_Schottky, symbol Device:D_Schottky
- removed R301: 0 DNP, symbol Device:R_Small
- added D301: 2SS100L-W, receiver-footprints:Rectron_SOD-123FL, symbol Device:D_Schottky_Small
- D302: Mouser (none) -> 583-2SS100L-W
- D303: footprint (none) -> receiver-footprints:Rectron_SOD-123FL
- D304: footprint (none) -> receiver-footprints:TI_X1SON; Mouser (none) -> 595-TPD1E04U04DPYR
- R302, R305: value 0 DNP -> 0
- R311: value 100k DNP -> 100k
- R314: footprint (none) -> Resistors_SMD:R_0402; Mouser (none) -> 603-RC0402JR-7D330RL
- R318: value 10k DNP -> 10k
Connections:
- net +3V3_ATTINY is gone; now on net +3V3: C304.1, J303.3 (Pin_3), U301.1 (VDD)
- net +3V3: now also D301.2 (A)
- net +5V_USB: now also D301.1 (K)
Other:
- note added: "DNP"
- moved on the sheet: C304
Changed lines of the file:
@@
 Wire Wire Line
 	9100 1700 8350 1700
-Text Label 3950 5700 2    50   ~ 0
+Text Label 4700 5700 2    50   ~ 0
 +3V3
 Text HLabel 4750 5800 0    50   Input ~ 0
@@
 L Device:C_Small C304
 U 1 1 5C040866
-P 4750 5500
-F 0 "C304" H 4760 5570 50  0000 L CNN
-F 1 "100 nF" H 4760 5420 50  0000 L CNN
-F 2 "Capacitors_SMD:C_0603_HandSoldering" H 4750 5500 50  0001 C CNN
-F 3 "~" H 4750 5500 50  0001 C CNN
-F 4 "710-885012206071" H 4750 5500 50  0001 C CNN "Mouser"
-	1    4750 5500
-	1    0    0    1
+P 4200 5700
+F 0 "C304" H 4210 5770 50  0000 L CNN
+F 1 "100 nF" H 4210 5620 50  0000 L CNN
+F 2 "Capacitors_SMD:C_0603_HandSoldering" H 4200 5700 50  0001 C CNN
+F 3 "~" H 4200 5700 50  0001 C CNN
+F 4 "710-885012206071" H 4200 5700 50  0001 C CNN "Mouser"
+	1    4200 5700
+	0    1    -1   0
 $EndComp
 $Comp
 L power:GND #PWR0125
 U 1 1 5C0408E6
-P 4750 5350
-F 0 "#PWR0125" H 4750 5100 50  0001 C CNN
-F 1 "GND" H 4750 5200 50  0000 C CNN
-F 2 "" H 4750 5350 50  0001 C CNN
-F 3 "" H 4750 5350 50  0001 C CNN
-	1    4750 5350
-	-1   0    0    1
-$EndComp
-Wire Wire Line
-	4750 5350 4750 5400
-Wire Wire Line
-	4750 5600 4750 5700
-Wire Wire Line
-	4750 5700 4850 5700
+P 4050 5700
+F 0 "#PWR0125" H 4050 5450 50  0001 C CNN
+F 1 "GND" H 4050 5550 50  0000 C CNN
+F 2 "" H 4050 5700 50  0001 C CNN
+F 3 "" H 4050 5700 50  0001 C CNN
+	1    4050 5700
+	0    1    1    0
+$EndComp
+Wire Wire Line
+	4050 5700 4100 5700
 Wire Wire Line
 	8450 1900 8350 1900
@@
 P 1950 3050
 F 0 "R302" H 1980 3070 50  0000 L CNN
-F 1 "0 DNP" H 1980 3010 50  0000 L CNN
+F 1 "0" H 1980 3010 50  0000 L CNN
 F 2 "" H 1950 3050 50  0001 C CNN
 F 3 "~" H 1950 3050 50  0001 C CNN
@@
 P 1950 3550
 F 0 "R305" H 1980 3570 50  0000 L CNN
-F 1 "0 DNP" H 1980 3510 50  0000 L CNN
+F 1 "0" H 1980 3510 50  0000 L CNN
 F 2 "" H 1950 3550 50  0001 C CNN
 F 3 "~" H 1950 3550 50  0001 C CNN
@@
 Wire Wire Line
 	6250 5800 6600 5800
-$Comp
-L Device:D_Schottky D301
-U 1 1 5C0716B1
-P 4250 5700
-F 0 "D301" H 4250 5800 50  0000 C CNN
-F 1 "D_Schottky" H 4250 5600 50  0000 C CNN
-F 2 "" H 4250 5700 50  0001 C CNN
-F 3 "~" H 4250 5700 50  0001 C CNN
-	1    4250 5700
-	-1   0    0    1
-$EndComp
-Wire Wire Line
-	3950 5700 4100 5700
-Wire Wire Line
-	4400 5700 4500 5700
-Connection ~ 4750 5700
-$Comp
-L Device:R_Small R301
-U 1 1 5C07590C
-P 4250 5500
-F 0 "R301" H 4280 5520 50  0000 L CNN
-F 1 "0 DNP" H 4280 5460 50  0000 L CNN
-F 2 "" H 4250 5500 50  0001 C CNN
-F 3 "~" H 4250 5500 50  0001 C CNN
-	1    4250 5500
-	0    1    -1   0
-$EndComp
-Wire Wire Line
-	4150 5500 3950 5500
-Wire Wire Line
-	3950 5500 3950 5700
-Wire Wire Line
-	4350 5500 4500 5500
-Wire Wire Line
-	4500 5500 4500 5700
-Connection ~ 4500 5700
-Wire Wire Line
-	4500 5700 4750 5700
 Text HLabel 6600 5800 2    50   Input ~ 0
 GAIN_SEL
@@
 P 7550 4550
 F 0 "R311" H 7580 4570 50  0000 L CNN
-F 1 "100k DNP" H 7580 4510 50  0000 L CNN
+F 1 "100k" H 7580 4510 50  0000 L CNN
 F 2 "" H 7550 4550 50  0001 C CNN
 F 3 "~" H 7550 4550 50  0001 C CNN
@@
 F 2 "" V 4750 3000 50  0001 C CNN
 F 3 "~" V 4750 3000 50  0001 C CNN
+F 4 "583-2SS100L-W" H 4750 3000 50  0001 C CNN "Mouser"
 	1    4750 3000
 	0    1    1    0
@@
 F 0 "D303" H 4700 3680 50  0000 L CNN
 F 1 "2SS100L-W" H 4470 3520 50  0000 L CNN
-F 2 "" V 4750 3600 50  0001 C CNN
+F 2 "receiver-footprints:Rectron_SOD-123FL" V 4750 3600 50  0001 C CNN
 F 3 "~" V 4750 3600 50  0001 C CNN
 	1    4750 3600
@@
 F 0 "R314" H 10530 5220 50  0000 L CNN
 F 1 "330" H 10530 5160 50  0000 L CNN
-F 2 "" H 10500 5200 50  0001 C CNN
+F 2 "Resistors_SMD:R_0402" H 10500 5200 50  0001 C CNN
 F 3 "~" H 10500 5200 50  0001 C CNN
+F 4 "603-RC0402JR-7D330RL" H 10500 5200 50  0001 C CNN "Mouser"
 	1    10500 5200
 	0    -1   -1   0
@@
 Wire Wire Line
 	10600 5300 10700 5300
-Text Label 4500 5500 1    50   ~ 0
-+3V3_ATTINY
-Text Label 10150 4700 2    50   ~ 0
-+3V3_ATTINY
-Wire Wire Line
-	10150 4700 10250 4700
 Text Label 10150 4600 2    50   ~ 0
 UPDI
@@
 F 0 "D304" H 9700 3730 50  0000 L CNN
 F 1 "TPD1E04U04DPYR" H 9600 3570 50  0000 L CNN
-F 2 "" V 9750 3650 50  0001 C CNN
+F 2 "receiver-footprints:TI_X1SON" V 9750 3650 50  0001 C CNN
 F 3 "~" V 9750 3650 50  0001 C CNN
+F 4 "595-TPD1E04U04DPYR" H 9750 3650 50  0001 C CNN "Mouser"
 	1    9750 3650
 	0    -1   1    0
@@
 $EndComp
 Wire Wire Line
-	2850 5750 2550 5750
+	2850 5750 2600 5750
 $Comp
 L Device:C_Small C320
@@
 Connection ~ 1550 5750
 Wire Wire Line
-	1550 5750 1650 5750
+	1550 5750 1600 5750
 $Comp
 L Device:C_Small C321
@@
 Wire Wire Line
 	2850 5850 2850 5750
-Text Notes 1650 5450 0    50   ~ 0
+Text Notes 1800 5200 0    50   ~ 0
 + 6 mA quiescent
-$Comp
-L power:PWR_FLAG #FLG0110
-U 1 1 5C4FB5FD
-P 10250 4750
-F 0 "#FLG0110" H 10250 4825 50  0001 C CNN
-F 1 "PWR_FLAG" H 10250 4900 50  0000 C CNN
-F 2 "" H 10250 4750 50  0001 C CNN
-F 3 "~" H 10250 4750 50  0001 C CNN
-	1    10250 4750
-	-1   0    0    1
-$EndComp
-Wire Wire Line
-	10250 4750 10250 4700
-Connection ~ 10250 4700
-Wire Wire Line
-	10250 4700 10700 4700
 $Comp
 L power:PWR_FLAG #FLG0111
@@
 P 2850 700
 F 0 "R318" H 2880 720 50  0000 L CNN
-F 1 "10k DNP" H 2880 660 50  0000 L CNN
+F 1 "10k" H 2880 660 50  0000 L CNN
 F 2 "" H 2850 700 50  0001 C CNN
 F 3 "~" H 2850 700 50  0001 C CNN
@@
 Wire Wire Line
 	2100 6050 2100 6150
+Text Notes 1800 2800 0    50   ~ 0
+DNP
+Text Notes 2100 3650 0    50   ~ 0
+DNP
+Text Notes 7700 4750 0    50   ~ 0
+DNP
+Text Notes 3000 800  0    50   ~ 0
+DNP
+$Comp
+L Device:D_Schottky_Small D301
+U 1 1 5C0DFE5D
+P 2150 5400
+F 0 "D301" H 2100 5480 50  0000 L CNN
+F 1 "2SS100L-W" H 1870 5320 50  0000 L CNN
+F 2 "receiver-footprints:Rectron_SOD-123FL" V 2150 5400 50  0001 C CNN
+F 3 "~" V 2150 5400 50  0001 C CNN
+	1    2150 5400
+	1    0    0    -1
+$EndComp
+Wire Wire Line
+	2250 5400 2600 5400
+Wire Wire Line
+	2600 5400 2600 5750
+Connection ~ 2600 5750
+Wire Wire Line
+	2600 5750 2550 5750
+Wire Wire Line
+	2050 5400 1600 5400
+Wire Wire Line
+	1600 5400 1600 5750
+Connection ~ 1600 5750
+Wire Wire Line
+	1600 5750 1650 5750
+Text Label 10150 4700 2    50   ~ 0
++3V3
+Wire Wire Line
+	10150 4700 10700 4700
+Wire Wire Line
+	4300 5700 4850 5700
 $EndSCHEMATC
