File: pcb/transmitter/controller.kicad_pcb (KiCad board)
At the start: 2 copper layers, 60 x 10 mm, 49 parts, among them J1 Conn_01x01, J2 Conn_01x02, J3 Conn_01x03, J4 Conn_02x02_Odd_Even, Q1 DMP3099L-7, Q3 BC847BLT1G, U1 TPS613222ADBVR, U2 LIS2DE12TR, U3 MSP430FR2512IRHLR, U4 BMG250, U5 TPS22917DBVR, Y1 32.786kHz

Commit message: Finish silkscreen layout
Parts:
- removed R103, R104: 33, Resistors_SMD:R_0603_HandSoldering
- removed R105: 47k, Resistors_SMD:R_0603_HandSoldering
- added R13: 33, Resistors_SMD:R_0603_HandSoldering, F.Cu at (48.8, 58.4)
- added R14: 33, Resistors_SMD:R_0603_HandSoldering, B.Cu at (77.0, 55.3)
- added R3: 47k, Resistors_SMD:R_0603_HandSoldering, F.Cu at (38.7, 56.3)
- renumbered C104 to C21
Routing:
- net /CAP: track 2.30 -> 2.82 mm

Commit message: Generate Gerbers
Routing:
- net GND: track 237.8 -> 241.6 mm, vias 23 -> 24
Changed lines of the file:
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@@
     (thickness 1.6)
     (drawings 20)
-    (tracks 599)
+    (tracks 610)
     (zones 0)
     (modules 49)
@@
   )
   (setup
-    (last_trace_width 0.254)
+    (last_trace_width 0.1524)
     (user_trace_width 0.1524)
     (user_trace_width 0.254)
@@
   (segment (start 53.844933 55.27) (end 53.854531 55.279598) (width 0.508) (layer F.Cu) (net 4))
   (segment (start 53.36 55.27) (end 53.844933 55.27) (width 0.508) (layer F.Cu) (net 4))
-  (via (at 52.45 54.59) (size 0.508) (drill 0.3302) (layers F.Cu B.Cu) (net 5))
+  (via (at 52.45 54.59) (size 0.508) (drill 0.3302) (layers F.Cu B.Cu) (net 5) (status 1000000))
   (segment (start 51.45 54.09) (end 51.95 54.09) (width 0.254) (layer F.Cu) (net 5))
   (segment (start 51.95 54.09) (end 52.45 54.59) (width 0.254) (layer F.Cu) (net 5))
@@
   (segment (start 55.45 54.619188) (end 55.45 52.89) (width 0.508) (layer F.Cu) (net 5))
   (segment (start 55.45 52.89) (end 62.00623 52.89) (width 0.254) (layer F.Cu) (net 5))
+  (via (at 51.52 51.7) (size 0.6858) (drill 0.3302) (layers F.Cu B.Cu) (net 5))
+  (segment (start 51.73 51.49) (end 51.52 51.7) (width 0.1524) (layer F.Cu) (net 5))
+  (segment (start 52.45 51.49) (end 51.73 51.49) (width 0.1524) (layer F.Cu) (net 5))
+  (segment (start 50.45 53.465) (end 50.45 53.69) (width 0.1524) (layer B.Cu) (net 5))
+  (segment (start 51.862899 52.052101) (end 50.45 53.465) (width 0.1524) (layer B.Cu) (net 5))
+  (segment (start 51.862899 52.042899) (end 51.862899 52.052101) (width 0.1524) (layer B.Cu) (net 5))
+  (segment (start 51.52 51.7) (end 51.862899 52.042899) (width 0.1524) (layer B.Cu) (net 5))
   (segment (start 53.5 53.49) (end 53.85 53.84) (width 0.254) (layer F.Cu) (net 6))
   (segment (start 52.45 53.49) (end 53.5 53.49) (width 0.254) (layer F.Cu) (net 6))
@@
   (segment (start 82.75 51.23079) (end 82.35921 50.84) (width 0.254) (layer F.Cu) (net 8))
   (segment (start 82.75 51.59) (end 82.75 51.23079) (width 0.254) (layer F.Cu) (net 8))
-  (segment (start 64.842094 52.027413) (end 72.416596 52.027413) (width 0.1524) (layer B.Cu) (net 8))
-  (segment (start 64.38165 51.207398) (end 64.632602 51.45835) (width 0.1524) (layer B.Cu) (net 8))
-  (segment (start 64.632602 51.45835) (end 64.632602 51.817921) (width 0.1524) (layer B.Cu) (net 8))
-  (segment (start 51.011756 51.207398) (end 64.38165 51.207398) (width 0.1524) (layer B.Cu) (net 8))
-  (segment (start 72.496001 51.948008) (end 72.75 51.694009) (width 0.1524) (layer B.Cu) (net 8))
-  (segment (start 72.416596 52.027413) (end 72.496001 51.948008) (width 0.1524) (layer B.Cu) (net 8))
-  (segment (start 64.632602 51.817921) (end 64.842094 52.027413) (width 0.1524) (layer B.Cu) (net 8))
   (via (at 50.369154 51.85) (size 0.6858) (drill 0.3302) (layers F.Cu B.Cu) (net 8))
-  (segment (start 50.369154 51.85) (end 51.011756 51.207398) (width 0.1524) (layer B.Cu) (net 8))
   (segment (start 48.81 52.7) (end 49.519154 52.7) (width 0.254) (layer F.Cu) (net 8))
   (segment (start 48.94 53.67) (end 48.94 52.83) (width 0.254) (layer B.Cu) (net 8))
@@
   (segment (start 48.62 52.89) (end 48.81 52.7) (width 0.254) (layer F.Cu) (net 8))
   (segment (start 47.51 52.89) (end 48.62 52.89) (width 0.254) (layer F.Cu) (net 8))
+  (segment (start 72.416596 52.027413) (end 72.496001 51.948008) (width 0.1524) (layer B.Cu) (net 8))
+  (segment (start 64.632602 51.817921) (end 64.842094 52.027413) (width 0.1524) (layer B.Cu) (net 8))
+  (segment (start 50.369154 51.85) (end 51.090655 51.128499) (width 0.1524) (layer B.Cu) (net 8))
+  (segment (start 72.496001 51.948008) (end 72.75 51.694009) (width 0.1524) (layer B.Cu) (net 8))
+  (segment (start 64.842094 52.027413) (end 72.416596 52.027413) (width 0.1524) (layer B.Cu) (net 8))
+  (segment (start 51.87322 51.207398) (end 64.38165 51.207398) (width 0.1524) (layer B.Cu) (net 8))
+  (segment (start 64.632602 51.45835) (end 64.632602 51.817921) (width 0.1524) (layer B.Cu) (net 8))
+  (segment (start 64.38165 51.207398) (end 64.632602 51.45835) (width 0.1524) (layer B.Cu) (net 8))
+  (segment (start 51.794321 51.128499) (end 51.87322 51.207398) (width 0.1524) (layer B.Cu) (net 8))
+  (segment (start 51.090655 51.128499) (end 51.794321 51.128499) (width 0.1524) (layer B.Cu) (net 8))
   (segment (start 46.714106 51.831894) (end 46.792099 51.831894) (width 0.254) (layer F.Cu) (net 9))
   (segment (start 46.61 52.49) (end 46.61 51.936) (width 0.254) (layer F.Cu) (net 9))
@@
   (segment (start 46.940205 51.98) (end 46.792099 51.831894) (width 0.254) (layer F.Cu) (net 9))
   (segment (start 48.18 51.98) (end 46.940205 51.98) (width 0.254) (layer F.Cu) (net 9))
-  (segment (start 66.116586 50.902587) (end 66.25 51.036001) (width 0.1524) (layer B.Cu) (net 9))
-  (segment (start 46.792099 51.831894) (end 47.721406 50.902587) (width 0.1524) (layer B.Cu) (net 9))
-  (segment (start 47.721406 50.902587) (end 66.116586 50.902587) (width 0.1524) (layer B.Cu) (net 9))
   (segment (start 81.025401 58.319401) (end 81 58.294) (width 0.254) (layer B.Cu) (net 9))
   (segment (start 74.4 51.29) (end 74.653999 51.036001) (width 0.254) (layer B.Cu) (net 9))
@@
   (segment (start 83.03206 51.036001) (end 84 52.003941) (width 0.254) (layer B.Cu) (net 9))
   (segment (start 83.770599 58.319401) (end 81.025401 58.319401) (width 0.254) (layer B.Cu) (net 9))
+  (segment (start 51.920577 50.823688) (end 51.999476 50.902587) (width 0.1524) (layer B.Cu) (net 9))
+  (segment (start 47.800305 50.823688) (end 51.920577 50.823688) (width 0.1524) (layer B.Cu) (net 9))
+  (segment (start 46.792099 51.831894) (end 47.800305 50.823688) (width 0.1524) (layer B.Cu) (net 9))
+  (segment (start 66.116586 50.902587) (end 66.25 51.036001) (width 0.1524) (layer B.Cu) (net 9))
+  (segment (start 51.999476 50.902587) (end 66.116586 50.902587) (width 0.1524) (layer B.Cu) (net 9))
   (via (at 66.9 51.09) (size 0.508) (drill 0.3302) (layers F.Cu B.Cu) (net 10))
   (segment (start 66.95 51.84) (end 66.95 51.14) (width 0.1524) (layer F.Cu) (net 10))
@@
   (segment (start 37.3 52.71) (end 37.32 52.73) (width 0.508) (layer F.Cu) (net 44))
   (segment (start 35.32 52.71) (end 37.3 52.71) (width 0.508) (layer F.Cu) (net 44))
-  (via (at 38.705518 52.890119) (size 0.6858) (drill 0.3302) (layers F.Cu B.Cu) (net 47))
-  (segment (start 39.685399 53.87) (end 40.11 53.87) (width 0.1524) (layer B.Cu) (net 47))
-  (segment (start 38.705518 52.890119) (end 39.685399 53.87) (width 0.1524) (layer B.Cu) (net 47))
-  (segment (start 38.705518 54.349518) (end 38.986 54.63) (width 0.254) (layer F.Cu) (net 47))
-  (segment (start 38.986 54.63) (end 40.02 54.63) (width 0.254) (layer F.Cu) (net 47))
-  (segment (start 38.705518 52.890119) (end 38.705518 54.349518) (width 0.254) (layer F.Cu) (net 47))
   (segment (start 82.25 53.64) (end 83.05 54.44) (width 0.254) (layer F.Cu) (net 46))
   (segment (start 81.3625 53.64) (end 82.25 53.64) (width 0.254) (layer F.Cu) (net 46))
@@
   (segment (start 80.6 51.665) (end 80.979 51.286) (width 0.254) (layer F.Cu) (net 46))
   (segment (start 82.127698 53.117698) (end 82.25 53.24) (width 0.254) (layer F.Cu) (net 46))
+  (via (at 38.705518 52.890119) (size 0.6858) (drill 0.3302) (layers F.Cu B.Cu) (net 47))
+  (segment (start 39.685399 53.87) (end 40.11 53.87) (width 0.1524) (layer B.Cu) (net 47))
+  (segment (start 38.705518 52.890119) (end 39.685399 53.87) (width 0.1524) (layer B.Cu) (net 47))
+  (segment (start 38.705518 54.349518) (end 38.986 54.63) (width 0.254) (layer F.Cu) (net 47))
+  (segment (start 38.986 54.63) (end 40.02 54.63) (width 0.254) (layer F.Cu) (net 47))
+  (segment (start 38.705518 52.890119) (end 38.705518 54.349518) (width 0.254) (layer F.Cu) (net 47))
   (zone (net 5) (net_name GND) (layer F.Cu) (hatch edge 0.508)
     (connect_pads (clearance 0.508))
